File: address_decoder.kicad_sch (KiCad schematic)
At the start: 56 parts, among them U17 74LS138, U18 74LS20

Commit message: chore: sync files
Parts:
- added U68: 74LS00, Package_DIP:DIP-14_W7.62mm_Socket, symbol 74xx:74LS00
- D65, D66, D67, D68, D69, D70, D71, D72, D73, D74, D75, D76, D77, D78, D79, D80, D81, D82, D83: footprint (none) -> LED_SMD:LED_0805_2012Metric
- R100, R65, R66, R67, R69, R70, R71, R72, R73, R74, R75, R76, R77, R78, R79, R80, R81, R82, R83, R84, R85, R86, R87, R88, R89, R90, R91, R92, R93, R94, R95, R96, R97, R98, R99: footprint (none) -> Resistor_SMD:R_0805_2012Metric
- U17: footprint (none) -> Package_DIP:DIP-16_W7.62mm_Socket
- U18: footprint (none) -> Package_DIP:DIP-14_W7.62mm_Socket
Connections:
- net +5V: now also U68.14 (VCC)
- net GND: now also U68.7 (GND)
- net at U17.10 (O5): now also U68.4
- new net: U68.10, U68.6, U68.9
- new net: U68.3, U68.5
- new net LCD_E: U68.8
- new net ~{RAM_I}: U68.1, U68.2
- no-connect marks 7 -> 6
Other:
- note added: "0xA00x Strobe 0xA001 LCD_RS"
- note added: "LCD"
