File: register_a.kicad_sch (KiCad schematic)
At the start: 18 parts, among them U24 74LS573, U25 74LS245

Commit message: chore: sync files
Parts:
- added U71: 74LS08, Package_DIP:DIP-14_W7.62mm_Socket, symbol 74xx:74LS08
- D100, D93, D94, D95, D96, D97, D98, D99: footprint (none) -> LED_SMD:LED_0805_2012Metric
- R109, R110, R111, R112, R113, R114, R115, R116: footprint (none) -> Resistor_SMD:R_0805_2012Metric
- U24, U25: footprint (none) -> Package_DIP:DIP-20_W7.62mm_Socket
Connections:
- net +5V: now also U71.14 (VCC)
- net GND: now also U71.7 (GND)
- net REG_A_I: now also U71.1; no longer U24.11 (Load)
- new net: U24.11 (Load), U71.3
- new net CLK: U71.2
Other:
- moved on the sheet: D100, D93, D94, D95, D96, D97, D98, D99, R109, R110, R111, R112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
