File: register_b_c.kicad_sch (KiCad schematic)
At the start: 37 parts, among them U1 74LS573, U2 74LS573, U3 74LS245, U4 74LS245, U70 74LS08

Commit message: chore: sync files
Parts:
- removed D1, D10, D11, D12, D13, D14, D15, D16, D2, D3, D4, D5, D6, D7, D8, D9: LED, LED_SMD:LED_0805_2012Metric, symbol Device:LED
- removed R1, R10, R11, R12, R13, R14, R15, R16, R2, R3, R4, R5, R6, R7, R8, R9: 470, Resistor_SMD:R_0805_2012Metric, symbol Device:R
- removed U1, U2: 74LS573, Package_DIP:DIP-20_W7.62mm_Socket, symbol 74xx:74LS573
- removed U3, U4: 74LS245, Package_DIP:DIP-20_W7.62mm_Socket, symbol 74xx:74LS245
- removed U70: 74LS08, Package_DIP:DIP-14_W7.62mm_Socket, symbol 74xx:74LS08
- added D133, D134, D135, D136, D137, D138, D139, D140, D141, D142, D143, D144, D145, D146, D147, D148: LED, LED_SMD:LED_0805_2012Metric, symbol Device:LED
- added R149, R150, R151, R152, R153, R154, R155, R156, R157, R158, R159, R160, R161, R162, R163, R164: 470, Resistor_SMD:R_0805_2012Metric, symbol Device:R
- added U36, U38: 74LS573, Package_DIP:DIP-20_W7.62mm_Socket, symbol 74xx:74LS573
- added U37, U39, U40, U41: 74LS245, Package_DIP:DIP-20_W7.62mm_Socket, symbol 74xx:74LS245
- added U73: 74LS08, Package_DIP:DIP-14_W7.62mm_Socket, symbol 74xx:74LS08
Connections:
- net +5V: now also U36.20 (VCC), U37.1 (A->B), U37.20 (VCC), U38.20 (VCC), U39.1 (A->B), U39.20 (VCC), U40.1 (A->B), U40.20 (VCC), U41.1 (A->B), U41.20 (VCC), U73.14 (VCC)
- net ADDR_BUS_0: now also U40.18 (B0)
- net ADDR_BUS_1: now also U40.17 (B1)
- net ADDR_BUS_10: now also U41.16 (B2)
- net ADDR_BUS_11: now also U41.15 (B3)
- net ADDR_BUS_12: now also U41.14 (B4)
- net ADDR_BUS_13: now also U41.13 (B5)
- net ADDR_BUS_14: now also U41.12 (B6)
- net ADDR_BUS_15: now also U41.11 (B7)
- net ADDR_BUS_2: now also U40.16 (B2)
- net ADDR_BUS_3: now also U40.15 (B3)
- net ADDR_BUS_4: now also U40.14 (B4)
- net ADDR_BUS_5: now also U40.13 (B5)
- net ADDR_BUS_6: now also U40.12 (B6)
- net ADDR_BUS_7: now also U40.11 (B7)
- net ADDR_BUS_8: now also U41.18 (B0)
- net ADDR_BUS_9: now also U41.17 (B1)
- net BUS_0: now also U36.2 (D0), U37.18 (B0), U38.2 (D0), U39.18 (B0)
- net BUS_1: now also U36.3 (D1), U37.17 (B1), U38.3 (D1), U39.17 (B1)
- net BUS_2: now also U36.4 (D2), U37.16 (B2), U38.4 (D2), U39.16 (B2)
- net BUS_3: now also U36.5 (D3), U37.15 (B3), U38.5 (D3), U39.15 (B3)
- net BUS_4: now also U36.6 (D4), U37.14 (B4), U38.6 (D4), U39.14 (B4)
- net BUS_5: now also U36.7 (D5), U37.13 (B5), U38.7 (D5), U39.13 (B5)
- net BUS_6: now also U36.8 (D6), U37.12 (B6), U38.8 (D6), U39.12 (B6)
- net BUS_7: now also U36.9 (D7), U37.11 (B7), U38.9 (D7), U39.11 (B7)
- net CLK: now also U73.2, U73.5
- net GND: now also D133.1 (K), D134.1 (K), D135.1 (K), D136.1 (K), D137.1 (K), D138.1 (K), D139.1 (K), D140.1 (K), D141.1 (K), D142.1 (K), D143.1 (K), D144.1 (K), D145.1 (K), D146.1 (K), D147.1 (K), D148.1 (K), U36.1 (OE), U36.10 (GND), U37.10 (GND), U38.1 (OE), U38.10 (GND), U39.10 (GND), U40.10 (GND), U41.10 (GND), U73.7 (GND)
- new net: R156.1, U36.19 (Q0), U37.2 (A0), U40.2 (A0)
- new net: R155.1, U36.18 (Q1), U37.3 (A1), U40.3 (A1)
- new net: R154.1, U36.17 (Q2), U37.4 (A2), U40.4 (A2)
- new net: R153.1, U36.16 (Q3), U37.5 (A3), U40.5 (A3)
- new net: R152.1, U36.15 (Q4), U37.6 (A4), U40.6 (A4)
- new net: R151.1, U36.14 (Q5), U37.7 (A5), U40.7 (A5)
- new net: R150.1, U36.13 (Q6), U37.8 (A6), U40.8 (A6)
- new net: R149.1, U36.12 (Q7), U37.9 (A7), U40.9 (A7)
- new net: D138.2 (A), R154.2
- new net: D139.2 (A), R155.2
- new net: D134.2 (A), R150.2
- new net: D147.2 (A), R163.2
- new net: D135.2 (A), R151.2
- new net: D144.2 (A), R160.2
- new net: D140.2 (A), R156.2
- new net: R157.1, U38.12 (Q7), U39.9 (A7), U41.9 (A7)
- new net: D141.2 (A), R157.2
- new net: U38.11 (Load), U73.6
- new net: R158.1, U38.13 (Q6), U39.8 (A6), U41.8 (A6)
- new net: R159.1, U38.14 (Q5), U39.7 (A5), U41.7 (A5)
- new net: R160.1, U38.15 (Q4), U39.6 (A4), U41.6 (A4)
- new net: R161.1, U38.16 (Q3), U39.5 (A3), U41.5 (A3)
- new net: R162.1, U38.17 (Q2), U39.4 (A2), U41.4 (A2)
- new net: R163.1, U38.18 (Q1), U39.3 (A1), U41.3 (A1)
- new net: R164.1, U38.19 (Q0), U39.2 (A0), U41.2 (A0)
- new net: D143.2 (A), R159.2
- new net: D148.2 (A), R164.2
- new net: D136.2 (A), R152.2
- new net: D142.2 (A), R158.2
- new net: D137.2 (A), R153.2
- new net: D146.2 (A), R162.2
- new net: D133.2 (A), R149.2
- new net: D145.2 (A), R161.2
- new net: U36.11 (Load), U73.3
- new net REG_B_I: U73.1
- new net REG_C_I: U73.4
- new net ~{PAIR_BC_O}: U40.19 (CE), U41.19 (CE)
- new net ~{REG_B_O}: U37.19 (CE)
- new net ~{REG_C_O}: U39.19 (CE)
Other:
- note removed: "MAR_H"
- note removed: "MAR_L"
- note removed: "Note that the LED part is optional, use the ~{OE} pins on the 573 and DNP LED and the 245 to save cost."
