File: register_d_e.kicad_sch (KiCad schematic)
At the start: 37 parts, among them U1 74LS573, U2 74LS573, U3 74LS245, U4 74LS245, U70 74LS08

Commit message: chore: sync files
Parts:
- removed D1, D10, D11, D12, D13, D14, D15, D16, D2, D3, D4, D5, D6, D7, D8, D9: LED, LED_SMD:LED_0805_2012Metric, symbol Device:LED
- removed R1, R10, R11, R12, R13, R14, R15, R16, R2, R3, R4, R5, R6, R7, R8, R9: 470, Resistor_SMD:R_0805_2012Metric, symbol Device:R
- removed U1, U2: 74LS573, Package_DIP:DIP-20_W7.62mm_Socket, symbol 74xx:74LS573
- removed U3, U4: 74LS245, Package_DIP:DIP-20_W7.62mm_Socket, symbol 74xx:74LS245
- removed U70: 74LS08, Package_DIP:DIP-14_W7.62mm_Socket, symbol 74xx:74LS08
- added D149, D150, D151, D152, D153, D154, D155, D156, D157, D158, D159, D160, D161, D162, D163, D164: LED, LED_SMD:LED_0805_2012Metric, symbol Device:LED
- added R165, R166, R167, R168, R169, R170, R171, R172, R173, R174, R175, R176, R177, R178, R179, R180: 470, Resistor_SMD:R_0805_2012Metric, symbol Device:R
- added U42, U43: 74LS573, Package_DIP:DIP-20_W7.62mm_Socket, symbol 74xx:74LS573
- added U44, U45, U46, U47: 74LS245, Package_DIP:DIP-20_W7.62mm_Socket, symbol 74xx:74LS245
- added U74: 74LS08, Package_DIP:DIP-14_W7.62mm_Socket, symbol 74xx:74LS08
Connections:
- net +5V: now also U42.20 (VCC), U43.20 (VCC), U44.1 (A->B), U44.20 (VCC), U45.1 (A->B), U45.20 (VCC), U46.1 (A->B), U46.20 (VCC), U47.1 (A->B), U47.20 (VCC), U74.14 (VCC)
- net ADDR_BUS_0: now also U46.18 (B0)
- net ADDR_BUS_1: now also U46.17 (B1)
- net ADDR_BUS_10: now also U47.16 (B2)
- net ADDR_BUS_11: now also U47.15 (B3)
- net ADDR_BUS_12: now also U47.14 (B4)
- net ADDR_BUS_13: now also U47.13 (B5)
- net ADDR_BUS_14: now also U47.12 (B6)
- net ADDR_BUS_15: now also U47.11 (B7)
- net ADDR_BUS_2: now also U46.16 (B2)
- net ADDR_BUS_3: now also U46.15 (B3)
- net ADDR_BUS_4: now also U46.14 (B4)
- net ADDR_BUS_5: now also U46.13 (B5)
- net ADDR_BUS_6: now also U46.12 (B6)
- net ADDR_BUS_7: now also U46.11 (B7)
- net ADDR_BUS_8: now also U47.18 (B0)
- net ADDR_BUS_9: now also U47.17 (B1)
- net BUS_0: now also U42.2 (D0), U43.2 (D0), U44.18 (B0), U45.18 (B0)
- net BUS_1: now also U42.3 (D1), U43.3 (D1), U44.17 (B1), U45.17 (B1)
- net BUS_2: now also U42.4 (D2), U43.4 (D2), U44.16 (B2), U45.16 (B2)
- net BUS_3: now also U42.5 (D3), U43.5 (D3), U44.15 (B3), U45.15 (B3)
- net BUS_4: now also U42.6 (D4), U43.6 (D4), U44.14 (B4), U45.14 (B4)
- net BUS_5: now also U42.7 (D5), U43.7 (D5), U44.13 (B5), U45.13 (B5)
- net BUS_6: now also U42.8 (D6), U43.8 (D6), U44.12 (B6), U45.12 (B6)
- net BUS_7: now also U42.9 (D7), U43.9 (D7), U44.11 (B7), U45.11 (B7)
- net CLK: now also U74.2, U74.5
- net GND: now also D149.1 (K), D150.1 (K), D151.1 (K), D152.1 (K), D153.1 (K), D154.1 (K), D155.1 (K), D156.1 (K), D157.1 (K), D158.1 (K), D159.1 (K), D160.1 (K), D161.1 (K), D162.1 (K), D163.1 (K), D164.1 (K), U42.1 (OE), U42.10 (GND), U43.1 (OE), U43.10 (GND), U44.10 (GND), U45.10 (GND), U46.10 (GND), U47.10 (GND), U74.7 (GND)
- new net: D154.2 (A), R170.2
- new net: U42.11 (Load), U74.3
- new net: U43.11 (Load), U74.6
- new net: R166.1, U43.12 (Q7), U45.9 (A7), U47.9 (A7)
- new net: R168.1, U43.13 (Q6), U45.8 (A6), U47.8 (A6)
- new net: R170.1, U43.14 (Q5), U45.7 (A5), U47.7 (A5)
- new net: R172.1, U43.15 (Q4), U45.6 (A4), U47.6 (A4)
- new net: R174.1, U43.16 (Q3), U45.5 (A3), U47.5 (A3)
- new net: R176.1, U43.17 (Q2), U45.4 (A2), U47.4 (A2)
- new net: R178.1, U43.18 (Q1), U45.3 (A1), U47.3 (A1)
- new net: R180.1, U43.19 (Q0), U45.2 (A0), U47.2 (A0)
- new net: R173.1, U42.16 (Q3), U44.5 (A3), U46.5 (A3)
- new net: D157.2 (A), R173.2
- new net: D156.2 (A), R172.2
- new net: R177.1, U42.18 (Q1), U44.3 (A1), U46.3 (A1)
- new net: D161.2 (A), R177.2
- new net: D159.2 (A), R175.2
- new net: D149.2 (A), R165.2
- new net: D162.2 (A), R178.2
- new net: R165.1, U42.12 (Q7), U44.9 (A7), U46.9 (A7)
- new net: R169.1, U42.14 (Q5), U44.7 (A5), U46.7 (A5)
- new net: D153.2 (A), R169.2
- new net: R167.1, U42.13 (Q6), U44.8 (A6), U46.8 (A6)
- new net: R171.1, U42.15 (Q4), U44.6 (A4), U46.6 (A4)
- new net: R175.1, U42.17 (Q2), U44.4 (A2), U46.4 (A2)
- new net: R179.1, U42.19 (Q0), U44.2 (A0), U46.2 (A0)
- new net: D152.2 (A), R168.2
- new net: D163.2 (A), R179.2
- new net: D155.2 (A), R171.2
- new net: D164.2 (A), R180.2
- new net: D151.2 (A), R167.2
- new net: D158.2 (A), R174.2
- new net: D150.2 (A), R166.2
- new net: D160.2 (A), R176.2
- new net REG_D_I: U74.1
- new net REG_E_I: U74.4
- new net ~{PAIR_DE_O}: U46.19 (CE), U47.19 (CE)
- new net ~{REG_D_O}: U44.19 (CE)
- new net ~{REG_E_O}: U45.19 (CE)
Other:
- note removed: "MAR_H"
- note removed: "MAR_L"
- note removed: "Note that the LED part is optional, use the ~{OE} pins on the 573 and DNP LED and the 245 to save cost."
