File: register_h_l.kicad_sch (KiCad schematic)
At the start: 40 parts, among them U26 74LS193, U27 74LS193, U48 74LS193, U49 74LS193, U50 74LS245, U51 74LS245, U52 74LS245, U53 74LS245

Commit message: chore: add files for simulation
Other:
- note added: "investigate negated behaviour"
Changed lines of the file:
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@@
 	(generator_version "10.0")
 	(paper "A3")
+	(text "investigate negated behaviour"
+		(exclude_from_sim no)
+		(at 103.886 106.934 0)
+		(effects
+			(font
+				(size 1.27 1.27)
+			)
+		)
+	)
 	(junction
 		(at 190.5 104.14)
