File: 8bit.kicad_sch (KiCad schematic)
At the start: 0 parts

Commit message: chore: sync files
Other:
- removed sheet Register B
- added sheet Clock (clock.kicad_sch)
- added sheet Instruction Decoder (instruction_decoder.kicad_sch)
- added sheet Instruction Register (register_instruction.kicad_sch)
- added sheet LCD Output (lcd_driver.kicad_sch)
- added sheet Output Register (register_output.kicad_sch)
- added sheet Register pair BC (register_b_c.kicad_sch)
- added sheet Register pair DE (register_d_e.kicad_sch)
- added sheet Register pair HL (register_h_l.kicad_sch)
- added sheet Step Counter (step_counter.kicad_sch)
- sheet ALU ports: added ALU_B_I, ALU_M, ALU_S0, ALU_S1, ALU_S2, ALU_S3, A_REG_0, A_REG_1, A_REG_2, A_REG_3, A_REG_4, A_REG_5, A_REG_6, A_REG_7, BUS_0, BUS_1, BUS_2, BUS_3, BUS_4, BUS_5, BUS_6, BUS_7, CF, CLK, FR_I, NF, VF, ZF, ~{ALU_O}; removed none
- sheet Address Decoder ports: added ADDR_BUS_0, ADDR_BUS_1, ADDR_BUS_10, ADDR_BUS_11, ADDR_BUS_12, ADDR_BUS_13, ADDR_BUS_14, ADDR_BUS_15, ADDR_BUS_2, ADDR_BUS_3, ADDR_BUS_4, ADDR_BUS_5, ADDR_BUS_6, ADDR_BUS_7, ADDR_BUS_8, ADDR_BUS_9, LCD_E, LCD_RS, ~{CF_CS}, ~{RAM_CS}, ~{RAM_I}, ~{ROM_CS}; removed none
- sheet CF reader ports: added ADDR_BUS_0, ADDR_BUS_1, ADDR_BUS_2, BUS_0, BUS_1, BUS_2, BUS_3, BUS_4, BUS_5, BUS_6, BUS_7, ~{CF_CS}, ~{CF_RD}, ~{CF_WR}, ~{RST}; removed none
- sheet MAR ports: added ADDR_BUS_0, ADDR_BUS_1, ADDR_BUS_10, ADDR_BUS_11, ADDR_BUS_12, ADDR_BUS_13, ADDR_BUS_14, ADDR_BUS_15, ADDR_BUS_2, ADDR_BUS_3, ADDR_BUS_4, ADDR_BUS_5, ADDR_BUS_6, ADDR_BUS_7, ADDR_BUS_8, ADDR_BUS_9, BUS_0, BUS_1, BUS_2, BUS_3, BUS_4, BUS_5, BUS_6, BUS_7, CLK, MAR_H_I, MAR_L_I, ~{MAR_O}; removed none
- sheet Program Counter ports: added ADDR_BUS_0, ADDR_BUS_1, ADDR_BUS_10, ADDR_BUS_11, ADDR_BUS_12, ADDR_BUS_13, ADDR_BUS_14, ADDR_BUS_15, ADDR_BUS_2, ADDR_BUS_3, ADDR_BUS_4, ADDR_BUS_5, ADDR_BUS_6, ADDR_BUS_7, ADDR_BUS_8, ADDR_BUS_9, BUS_0, BUS_1, BUS_2, BUS_3, BUS_4, BUS_5, BUS_6, BUS_7, CLK, PC_E, ~{JMP_H}, ~{JMP_L}, ~{PC_O}, ~{RST}; removed none
- sheet RAM ports: added ADDR_BUS_0, ADDR_BUS_1, ADDR_BUS_10, ADDR_BUS_11, ADDR_BUS_12, ADDR_BUS_13, ADDR_BUS_14, ADDR_BUS_2, ADDR_BUS_3, ADDR_BUS_4, ADDR_BUS_5, ADDR_BUS_6, ADDR_BUS_7, ADDR_BUS_8, ADDR_BUS_9, BUS_0, BUS_1, BUS_2, BUS_3, BUS_4, BUS_5, BUS_6, BUS_7, ~{RAM_CS}, ~{RAM_I}; removed none
- sheet ROM ports: added ADDR_BUS_0, ADDR_BUS_1, ADDR_BUS_10, ADDR_BUS_11, ADDR_BUS_12, ADDR_BUS_2, ADDR_BUS_3, ADDR_BUS_4, ADDR_BUS_5, ADDR_BUS_6, ADDR_BUS_7, ADDR_BUS_8, ADDR_BUS_9, BUS_0, BUS_1, BUS_2, BUS_3, BUS_4, BUS_5, BUS_6, BUS_7, ~{ROM_CS}; removed none
- sheet Register A ports: added A_REG_0, A_REG_1, A_REG_2, A_REG_3, A_REG_4, A_REG_5, A_REG_6, A_REG_7, BUS_0, BUS_1, BUS_2, BUS_3, BUS_4, BUS_5, BUS_6, BUS_7, CLK, REG_A_I, ~{REG_A_O}; removed none
- sheet Stack Pointer ports: added ADDR_BUS_0, ADDR_BUS_1, ADDR_BUS_10, ADDR_BUS_11, ADDR_BUS_12, ADDR_BUS_13, ADDR_BUS_14, ADDR_BUS_15, ADDR_BUS_2, ADDR_BUS_3, ADDR_BUS_4, ADDR_BUS_5, ADDR_BUS_6, ADDR_BUS_7, ADDR_BUS_8, ADDR_BUS_9, BUS_0, BUS_1, BUS_2, BUS_3, BUS_4, BUS_5, BUS_6, BUS_7, RST, ~{POP}, ~{PUSH}, ~{SP_H_I}, ~{SP_L_I}, ~{SP_O}; removed none

Commit message: chore: sync design between simulation and schematic
Other:
- added sheet Misc (misc.kicad_sch)
- added sheet Temporary Register (register_temporary.kicad_sch)
- sheet ALU ports: added ALU_CARRY, ~{RAR_OUT}, ~{RRC_OUT}; removed none
- sheet Instruction Decoder ports: added none; removed BUS_0, BUS_1, BUS_2, BUS_3, BUS_4, BUS_5, BUS_6, BUS_7
- sheet MAR ports: added MAR_INC, PROG, ~{RST}; removed none
- sheet Program Counter ports: added ~{PC_B_HOUT}, ~{PC_B_LOUT}; removed none
- sheet RAM ports: added CLK, PROG, RAM_I, RAM_O; removed ~{RAM_I}
- sheet Stack Pointer ports: added CLK, SP_H_I; removed ~{SP_H_I}
- sheet Step Counter ports: added CLK, PROG; removed none
