File: alu.kicad_sch (KiCad schematic)
At the start: 56 parts, among them U28 74LS181, U29 74LS181, U30 74LS245, U31 74LS373, U32 74LS573, U33 74LS08, U34 74LS02, U35 74LS04

Commit message: chore: sync files
Parts:
- removed D125, D126, D127, D128: LED, symbol Device:LED
- removed R141, R142, R143, R144: 470, symbol Device:R
- added unit 2 of U35
- added U72 (x2): 74LS08, Package_DIP:DIP-14_W7.62mm_Socket, symbol 74xx:74LS08
- added U77: 74LS86, Package_DIP:DIP-14_W7.62mm_Socket, symbol 74xx:74LS86
- D109, D110, D111, D112, D113, D114, D115, D116, D117, D118, D119, D120, D121, D122, D123, D124, D129, D130, D131, D132: footprint (none) -> LED_SMD:LED_0805_2012Metric
- R125, R126, R127, R128, R129, R130, R131, R132, R133, R134, R135, R136, R137, R138, R139, R140, R145, R146, R147, R148: footprint (none) -> Resistor_SMD:R_0805_2012Metric
- U28, U29: footprint (none) -> Package_DIP:DIP-24_W15.24mm_Socket
- U30, U31, U32: footprint (none) -> Package_DIP:DIP-20_W7.62mm_Socket
- U33, U34, U35: footprint (none) -> Package_DIP:DIP-14_W7.62mm_Socket
Connections:
- net +5V: now also U72.14 (VCC), U77.14 (VCC)
- net ALU_B_I: now also U72.4; no longer U31.11 (LE)
- net A_REG_7: now also U77.2, U77.5
- net FR_I: now also U72.1; no longer U32.11 (Load)
- net GND: now also U72.7 (GND), U77.7 (GND)
- net VF: now reaches R145.1, U32.16 (Q3)
- net at U32.4 (D2): now also R125.1, U29.13 (F3), U30.9 (A7), U34.3, U77.4; no longer U29.14 (A=B)
- net at U32.5 (D3): now also U72.6
- net at R133.1, U29.18 (B3), U31.19 (O7): now also U77.1
- net EF renamed NF
- new net: U35.3, U77.3
- new net: U35.4, U72.5
- new net: U32.11 (Load), U72.3
- new net: U72.4, U77.6
- new net: U31.11 (LE), U72.6
- new net CLK: U72.2, U72.5
- no-connect marks 5 -> 14
Other:
- moved on the sheet: D129, D130, D131, D132, R145, R146, R147, R148, U34E, U35A, U35G

Commit message: chore: add files for simulation
Other:
- note added: "use 573 instead"
Changed lines of the file:
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@@
 	(generator_version "10.0")
 	(paper "A3")
+	(text "use 573 instead"
+		(exclude_from_sim no)
+		(at 92.71 101.854 0)
+		(effects
+			(font
+				(size 1.27 1.27)
+			)
+		)
+	)
 	(text "Flags Register"
 		(exclude_from_sim no)

Commit message: chore: sync design between simulation and schematic
Parts:
- removed U31: 74LS373, Package_DIP:DIP-20_W7.62mm_Socket, symbol 74xx:74LS373
- removed U72: 74LS08, Package_DIP:DIP-14_W7.62mm_Socket, symbol 74xx:74LS08
- added U31: 74LS245, Package_DIP:DIP-20_W7.62mm_Socket, symbol 74xx:74LS245
- added unit 3 of U35
- added unit 3 of U72
- added U75: 74LS08, Package_DIP:DIP-14_W7.62mm_Socket, symbol 74xx:74LS08
- added U96: 74LS573, symbol 74xx:74LS573
- added U97: 74LS157, symbol 74xx:74LS157
Connections:
- net +5V: now also U31.1 (A->B), U31.20 (VCC), U96.20 (VCC), U97.16 (VCC); no longer U28.7 (Cn)
- net ALU_B_I: now also U75.4
- net A_REG_0: now also U97.2 (I0a), U97.6 (I1b)
- net A_REG_1: now also U31.2 (A0)
- net A_REG_2: now also U31.3 (A1)
- net A_REG_3: now also U31.4 (A2)
- net A_REG_4: now also U31.5 (A3)
- net A_REG_5: now also U31.6 (A4)
- net A_REG_6: now also U31.7 (A5)
- net A_REG_7: now also U31.8 (A6)
- net BUS_0: now also U96.2 (D0)
- net BUS_1: now also U96.3 (D1)
- net BUS_2: now also U96.4 (D2)
- net BUS_3: now also U96.5 (D3)
- net BUS_4: now also U96.6 (D4)
- net BUS_5: now also U96.7 (D5)
- net BUS_6: now also U96.8 (D6)
- net BUS_7: now also U96.9 (D7)
- net CLK: now also U75.5
- net GND: now also U31.10 (GND), U96.1 (OE), U96.10 (GND), U97.15 (E), U97.8 (GND)
- net at R139.1, U28.22 (B1): now also U31.17 (B1), U96.18 (Q1)
- net at R137.1, U28.18 (B3): now also U31.15 (B3), U96.16 (Q3)
- net at U32.3 (D1): now also U97.4 (Za); no longer U35.2
- net at R133.1, U29.18 (B3), U77.1: now also U31.11 (B7), U96.12 (Q7)
- net at R136.1, U29.1 (B0): now also U31.14 (B4), U96.15 (Q4)
- net at R135.1, U29.22 (B1): now also U31.13 (B5), U96.14 (Q5)
- net at R134.1, U29.20 (B2): now also U31.12 (B6), U96.13 (Q6)
- net at R140.1, U28.1 (B0): now also U31.18 (B0), U96.19 (Q0)
- net at R138.1, U28.20 (B2): now also U31.16 (B2), U96.17 (Q2)
- new net: U31.19 (CE), U72.8
- new net: U75.6, U96.11 (Load)
- new net: U35.2, U97.3 (I1a)
- new net ALU_CARRY: U35.5, U97.5 (I0b)
- new net D8: U31.9 (A7), U97.7 (Zb)
- new net ~{ALU_CARRY}: U28.7 (Cn), U35.6
- new net ~{RAR_OUT}: U72.10, U97.1 (S)
- new net ~{RRC_OUT}: U72.9
- no-connect marks 14 -> 20
Other:
- note removed: "use 573 instead"
- moved on the sheet: D109, D110, D111, D112, D113, D114, D115, D116, D129, D130, D131, D132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
