File: mar.kicad_sch (KiCad schematic)
At the start: 37 parts, among them U1 74LS573, U2 74LS573, U3 74LS245, U4 74LS245, U70 74LS08

Commit message: chore: sync design between simulation and schematic
Parts:
- removed D1, D10, D11, D12, D13, D14, D15, D16, D2, D3, D4, D5, D6, D7, D8, D9: LED, LED_SMD:LED_0805_2012Metric, symbol Device:LED
- removed R1, R10, R11, R12, R13, R14, R15, R16, R2, R3, R4, R5, R7, R8, R9: 470, Resistor_SMD:R_0805_2012Metric, symbol Device:R
- removed U1, U2: 74LS573, Package_DIP:DIP-20_W7.62mm_Socket, symbol 74xx:74LS573
- removed U3, U4: 74LS245, Package_DIP:DIP-20_W7.62mm_Socket, symbol 74xx:74LS245
- removed U70: 74LS08, Package_DIP:DIP-14_W7.62mm_Socket, symbol 74xx:74LS08
- added D126, D127, D128, D185, D186, D187, D188, D189, D190, D191, D192, D193, D194, D195, D196, D197, D206: LED, LED_SMD:LED_0805_2012Metric, symbol Device:LED
- added R210, R211, R212, R213, R214, R215, R216, R217, R218, R219, R220, R221, R222, R223, R224, R225, R250: 470, Resistor_SMD:R_0805_2012Metric, symbol Device:R
- added R232, R233, R234, R235, R236, R237, R238, R239: 1k, Resistor_SMD:R_0805_2012Metric, symbol Device:R
- added SW4: SW_DIP_x08, symbol Switch:SW_DIP_x08
- added SW9: L/~{H}, symbol Switch:SW_SPDT
- added U1: 74LS04, symbol 74xx:74LS04
- added U2: 74LS08, symbol 74xx:74LS08
- added U3: 74LS32, symbol 74xx:74LS32
- added U84, U85, U86, U87: 74LS161, Package_DIP:DIP-16_W7.62mm_Socket, symbol 74xx:74LS161
- added U88, U89: 74LS245, Package_DIP:DIP-20_W7.62mm_Socket, symbol 74xx:74LS245
- added U90, U91: 74LS245, symbol 74xx:74LS245
- R6: value 470 -> 1k; footprint Resistor_SMD:R_0805_2012Metric -> (none)
Connections:
- net +5V: now also SW4.1, SW4.2, SW4.3, SW4.4, SW4.5, SW4.6, SW4.7, SW4.8, SW9.2 (B), U1.14 (VCC), U2.14 (VCC), U3.14 (VCC), U84.10 (CET), U84.16 (VCC), U85.16 (VCC), U86.16 (VCC), U87.16 (VCC), U88.1 (A->B), U88.20 (VCC), U89.1 (A->B), U89.20 (VCC), U90.1 (A->B), U90.20 (VCC), U91.1 (A->B), U91.20 (VCC)
- net ADDR_BUS_0: now also U88.18 (B0)
- net ADDR_BUS_1: now also U88.17 (B1)
- net ADDR_BUS_10: now also U89.16 (B2)
- net ADDR_BUS_11: now also U89.15 (B3)
- net ADDR_BUS_12: now also U89.14 (B4)
- net ADDR_BUS_13: now also U89.13 (B5)
- net ADDR_BUS_14: now also U89.12 (B6)
- net ADDR_BUS_15: now also U89.11 (B7)
- net ADDR_BUS_2: now also U88.16 (B2)
- net ADDR_BUS_3: now also U88.15 (B3)
- net ADDR_BUS_4: now also U88.14 (B4)
- net ADDR_BUS_5: now also U88.13 (B5)
- net ADDR_BUS_6: now also U88.12 (B6)
- net ADDR_BUS_7: now also U88.11 (B7)
- net ADDR_BUS_8: now also U89.18 (B0)
- net ADDR_BUS_9: now also U89.17 (B1)
- net BUS_0: now also U90.2 (A0)
- net BUS_1: now also U90.3 (A1)
- net BUS_2: now also U90.4 (A2)
- net BUS_3: now also U90.5 (A3)
- net BUS_4: now also U90.6 (A4)
- net BUS_5: now also U90.7 (A5)
- net BUS_6: now also U90.8 (A6)
- net BUS_7: now also U90.9 (A7)
- net CLK: now also U84.2 (CP), U85.2 (CP), U86.2 (CP), U87.2 (CP)
- net GND: now also R6.2, D126.1 (K), D127.1 (K), D128.1 (K), D185.1 (K), D186.1 (K), D187.1 (K), D188.1 (K), D189.1 (K), D190.1 (K), D191.1 (K), D192.1 (K), D193.1 (K), D194.1 (K), D195.1 (K), D196.1 (K), D197.1 (K), D206.1 (K), R232.2, R233.2, R234.2, R235.2, R236.2, R237.2, R238.2, R239.2, U1.7 (GND), U2.7 (GND), U3.7 (GND), U84.8 (GND), U85.8 (GND), U86.8 (GND), U87.8 (GND), U88.10 (GND), U89.10 (GND), U90.10 (GND), U91.10 (GND)
- net MAR_H_I: now also U3.4
- net MAR_L_I: now also U3.1
- net ~{MAR_O}: now also U3.10
- net at R6.1: now also R250.1, SW9.1 (A), U1.1, U2.2
- new net: D126.2 (A), R210.2
- new net: D189.2 (A), R217.2
- new net: R233.1, SW4.16, U91.2 (A0)
- new net: R210.1, U87.11 (Q3), U89.9 (A7)
- new net: D194.2 (A), R222.2
- new net: U2.3, U3.2
- new net: U3.3, U84.9 (~{PE}), U85.9 (~{PE})
- new net: D187.2 (A), R215.2
- new net: R211.1, U87.12 (Q2), U89.8 (A6)
- new net: D127.2 (A), R211.2
- new net: D192.2 (A), R220.2
- new net: D196.2 (A), R224.2
- new net: U85.6 (D3), U87.6 (D3), U90.11 (B7), U91.11 (B7)
- new net: U85.5 (D2), U87.5 (D2), U90.12 (B6), U91.12 (B6)
- new net: U85.4 (D1), U87.4 (D1), U90.13 (B5), U91.13 (B5)
- new net: U85.3 (D0), U87.3 (D0), U90.14 (B4), U91.14 (B4)
- new net: U84.6 (D3), U86.6 (D3), U90.15 (B3), U91.15 (B3)
- new net: U84.5 (D2), U86.5 (D2), U90.16 (B2), U91.16 (B2)
- new net: U84.4 (D1), U86.4 (D1), U90.17 (B1), U91.17 (B1)
- new net: U84.3 (D0), U86.3 (D0), U90.18 (B0), U91.18 (B0)
- new net: R223.1, U84.12 (Q2), U88.4 (A2)
- new net: D195.2 (A), R223.2
- new net: R221.1, U85.14 (Q0), U88.6 (A4)
- new net: D193.2 (A), R221.2
- new net: D190.2 (A), R218.2
- new net: U2.6, U3.5
- new net: U3.6, U86.9 (~{PE}), U87.9 (~{PE})
- new net: U3.8, U88.19 (CE), U89.19 (CE)
- new net: D206.2 (A), R250.2
- new net: R220.1, U85.13 (Q1), U88.7 (A5)
- new net: R238.1, SW4.10, U91.8 (A6)
- new net: R237.1, SW4.11, U91.7 (A5)
- new net: R236.1, SW4.12, U91.6 (A4)
- new net: R235.1, SW4.13, U91.5 (A3)
- new net: R234.1, SW4.14, U91.4 (A2)
- new net: R232.1, SW4.15, U91.3 (A1)
- new net: R239.1, SW4.9, U91.9 (A7)
- new net: R215.1, U86.12 (Q2), U89.4 (A2)
- new net: D197.2 (A), R225.2
- new net: D186.2 (A), R214.2
- new net: U1.2, U2.5
- new net: R218.1, U85.11 (Q3), U88.9 (A7)
- new net: D185.2 (A), R213.2
- new net: U84.15 (TC), U85.10 (CET)
- new net: R219.1, U85.12 (Q2), U88.8 (A6)
- new net: U85.15 (TC), U86.10 (CET)
- new net: R212.1, U87.13 (Q1), U89.7 (A5)
- new net: D128.2 (A), R212.2
- new net: U86.15 (TC), U87.10 (CET)
- new net: R213.1, U87.14 (Q0), U89.6 (A4)
- new net: R217.1, U86.14 (Q0), U89.2 (A0)
- new net: R224.1, U84.13 (Q1), U88.3 (A1)
- new net: R225.1, U84.14 (Q0), U88.2 (A0)
- new net: R222.1, U84.11 (Q3), U88.5 (A3)
- new net: D191.2 (A), R219.2
- new net: D188.2 (A), R216.2
- new net: R216.1, U86.13 (Q1), U89.3 (A1)
- new net: R214.1, U86.11 (Q3), U89.5 (A3)
- new net MAR_INC: U84.7 (CEP), U85.7 (CEP), U86.7 (CEP), U87.7 (CEP)
- new net PROG: U1.3, U2.1, U2.4
- new net ~{PROG}: U1.4, U3.9, U90.19 (CE), U91.19 (CE)
- new net ~{RST}: U84.1 (~{MR}), U85.1 (~{MR}), U86.1 (~{MR}), U87.1 (~{MR})
- no-connect marks 0 -> 2
Other:
- note added: "PC_H"
- note added: "PC_L"
- note removed: "MAR_H"
- note removed: "MAR_L"
- note removed: "Note that the LED part is optional, use the ~{OE} pins on the 573 and DNP LED and the 245 to save cost."
