File: schematic/8bit.kicad_sch (KiCad schematic)
At the start: 0 parts

Commit message: chore: sync outdated schematic files
Other:
- sheet Address Decoder ports: added RAM_I; removed ~{RAM_I}
- sheet Stack Pointer ports: added SP_L_I; removed ~{SP_L_I}

Commit message: feat: address decoding completed, general clean up
Connections:
- no-connect marks 0 -> 2
Other:
- sheet Instruction Decoder ports: added CTRL_WORDS; removed none
- sheet Register pair HL ports: added CLK, REG_H_I, REG_L_I; removed ~{REG_H_I}, ~{REG_L_I}
- note added: "TBD!!!"
