File: schematic/address_decoder.kicad_sch (KiCad schematic)
At the start: 57 parts, among them U17 74LS138, U18 74LS20, U68 74LS00

Commit message: chore: sync outdated schematic files
Parts:
- removed unit 1 of U68
Connections:
- net RAM_I: now reaches U68.5
Changed lines of the file:
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@@
 	(wire
 		(pts
-			(xy 214.63 144.78) (xy 214.63 149.86)
-		)
-		(stroke
-			(width 0)
-			(type default)
-		)
-	)
-	(wire
-		(pts
 			(xy 73.66 78.74) (xy 73.66 87.63)
 		)
@@
 	(wire
 		(pts
-			(xy 229.87 149.86) (xy 234.95 149.86)
+			(xy 231.14 149.86) (xy 234.95 149.86)
 		)
 		(stroke
@@
 	(wire
 		(pts
-			(xy 229.87 147.32) (xy 229.87 149.86)
-		)
-		(stroke
-			(width 0)
-			(type default)
-		)
-	)
-	(wire
-		(pts
 			(xy 88.9 100.33) (xy 93.98 100.33)
 		)
@@
 		)
 	)
-	(hierarchical_label "~{RAM_I}"
+	(hierarchical_label "RAM_I"
 		(shape input)
-		(at 214.63 147.32 180)
+		(at 231.14 149.86 180)
 		(effects
 			(font
@@
 					(unit 1)
 				)
-			)
-		)
-	)
-	(symbol
-		(lib_id "74xx:74LS00")
-		(at 222.25 147.32 0)
-		(unit 1)
-		(body_style 1)
-		(exclude_from_sim no)
-		(in_bom yes)
-		(on_board yes)
-		(in_pos_files yes)
-		(dnp no)
-		(fields_autoplaced yes)
-		(property "Reference" "U68"
-			(at 222.2417 138.43 0)
-			(show_name no)
-			(do_not_autoplace no)
-			(effects
-				(font
-					(size 1.27 1.27)
-				)
-			)
-		)
-		(property "Value" "74LS00"
-			(at 222.2417 140.97 0)
-			(show_name no)
-			(do_not_autoplace no)
-			(effects
-				(font
-					(size 1.27 1.27)
-				)
-			)
-		)
-		(property "Footprint" "Package_DIP:DIP-14_W7.62mm_Socket"
-			(at 222.25 147.32 0)
-			(hide yes)
-			(show_name no)
-			(do_not_autoplace no)
-			(effects
-				(font
-					(size 1.27 1.27)
-				)
-			)
-		)
-		(property "Datasheet" "http://www.ti.com/lit/gpn/sn74ls00"
-			(at 222.25 147.32 0)
-			(hide yes)
-			(show_name no)
-			(do_not_autoplace no)
-			(effects
-				(font
-					(size 1.27 1.27)
-				)
-			)
-		)
-		(property "Description" "quad 2-input NAND gate"
-			(at 222.25 147.32 0)
-			(hide yes)
-			(show_name no)
-			(do_not_autoplace no)
-			(effects
-				(font
-					(size 1.27 1.27)
-				)
-			)
-		)
-		(pin "11"
-		)
-		(pin "12"
-		)
-		(pin "13"
-		)
-		(pin "9"
-		)
-		(pin "10"
-		)
-		(pin "8"
-		)
-		(pin "2"
-		)
-		(pin "3"
-		)
-		(pin "1"
-		)
-		(pin "5"
-		)
-		(pin "4"
-		)
-		(pin "6"
-		)
-		(pin "14"
-		)
-		(pin "7"
-		)
-		(instances
-			(project "8bit"
-				(path "/ce6ef060-f4bd-4228-ab8d-5cf6f386dba1/966ea3a8-e5ca-459e-b420-1b20e623a8eb"
-					(reference "U68")
-					(unit 1)
-				)

Commit message: feat: address decoding completed, general clean up
Parts:
- renumbered D68 to D50, D69 to D51, D70 to D52, D71 to D53, D72 to D54, D73 to D55, D74 to D56, D75 to D57, D76 to D58, D77 to D59, D78 to D60, D79 to D61, D80 to D62, D81 to D63, D82 to D64, D83 to D65, D67 to D66, D66 to D67, D65 to D68, R69 to R59, R70 to R60, R71 to R61, R72 to R62, R73 to R63, R74 to R64, R75 to R65, R76 to R66, R77 to R67, R78 to R68, R79 to R69, R80 to R70, R81 to R71, R82 to R72, R83 to R73, R84 to R74, R85 to R75, R86 to R76, R87 to R77, R88 to R78, R89 to R79, R90 to R80, R91 to R81, R92 to R82, R93 to R83, R94 to R84, R95 to R85, R96 to R86, R97 to R87, R98 to R88, R99 to R89, R100 to R90, R67 to R91, R66 to R92, R65 to R93, U68 to U27, U18 to U28, U17 to U29
Connections:
- net LCD_E: now also U27.6; no longer U27.8
- net RAM_I: now also U27.2; no longer U27.5
- net at U29.10 (O5): now also U27.1; no longer U27.4
- new net: U27.3, U27.4, U27.5
