File: schematic/program_counter.kicad_sch (KiCad schematic)
At the start: 40 parts, among them U10 74LS245, U5 74LS161, U6 74LS161, U7 74LS161, U70 74LS245, U8 74LS161, U9 74LS245, U93 74LS245

Commit message: feat: address decoding completed, general clean up
Parts:
- renumbered D17 to D18, D18 to D19, D19 to D20, D20 to D21, D21 to D22, D22 to D23, D23 to D24, D24 to D25, D25 to D26, D26 to D27, D27 to D28, D28 to D29, D29 to D30, D30 to D31, D31 to D32, D32 to D33, R17 to R27, R18 to R28, R19 to R29, R20 to R30, R21 to R31, R22 to R32, R23 to R33, R24 to R34, R25 to R35, R26 to R36, R27 to R37, R28 to R38, R29 to R39, R30 to R40, R31 to R41, R32 to R42, U5 to U12, U6 to U13, U7 to U14, U8 to U15, U9 to U16, U10 to U17, U70 to U18, U93 to U19
