File: schematic/register_a.kicad_sch (KiCad schematic)
At the start: 19 parts, among them U24 74LS573, U25 74LS245, U71 74LS08

Commit message: feat: address decoding completed, general clean up
Parts:
- renumbered D99 to D100, D100 to D101, D93 to D94, D94 to D95, D95 to D96, D96 to D97, D97 to D98, D98 to D99, R109 to R129, R110 to R130, R111 to R131, R112 to R132, R113 to R133, R114 to R134, R115 to R135, R116 to R136, U71 to U38, U24 to U39, U25 to U40
Changed lines of the file:
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@@
 		(dnp no)
 		(fields_autoplaced yes)
-		(property "Reference" "#PWR075"
+		(property "Reference" "#PWR0117"
 			(at 205.74 54.61 0)
 			(hide yes)
@@
 			(project "8bit"
 				(path "/ce6ef060-f4bd-4228-ab8d-5cf6f386dba1/a913a341-ba12-46a1-b026-37d3a35c843c"
-					(reference "#PWR075")
+					(reference "#PWR0117")
 					(unit 1)
 				)
@@
 		(in_pos_files yes)
 		(dnp no)
-		(property "Reference" "#PWR074"
+		(property "Reference" "#PWR0116"
 			(at 187.96 85.09 0)
 			(hide yes)
@@
 			(project "8bit"
 				(path "/ce6ef060-f4bd-4228-ab8d-5cf6f386dba1/a913a341-ba12-46a1-b026-37d3a35c843c"
-					(reference "#PWR074")
+					(reference "#PWR0116")
 					(unit 1)
 				)
@@
 		(dnp no)
 		(fields_autoplaced yes)
-		(property "Reference" "#PWR0191"
+		(property "Reference" "#PWR0111"
 			(at 36.83 60.96 0)
 			(hide yes)
@@
 			(project "8bit"
 				(path "/ce6ef060-f4bd-4228-ab8d-5cf6f386dba1/a913a341-ba12-46a1-b026-37d3a35c843c"
-					(reference "#PWR0191")
+					(reference "#PWR0111")
 					(unit 1)
 				)
@@
 		(dnp no)
 		(fields_autoplaced yes)
-		(property "Reference" "#PWR067"
+		(property "Reference" "#PWR0113"
 			(at 99.06 54.61 0)
 			(hide yes)
@@
 			(project "8bit"
 				(path "/ce6ef060-f4bd-4228-ab8d-5cf6f386dba1/a913a341-ba12-46a1-b026-37d3a35c843c"
-					(reference "#PWR067")
+					(reference "#PWR0113")
 					(unit 1)
 				)
@@
 		(dnp no)
 		(fields_autoplaced yes)
-		(property "Reference" "U24"
+		(property "Reference" "U39"
 			(at 101.2033 50.8 0)
 			(show_name no)
@@
 			(project "8bit"
 				(path "/ce6ef060-f4bd-4228-ab8d-5cf6f386dba1/a913a341-ba12-46a1-b026-37d3a35c843c"
-					(reference "U24")
+					(reference "U39")
 					(unit 1)
 				)
@@
 		(in_pos_files yes)
 		(dnp no)
-		(property "Reference" "R115"
+		(property "Reference" "R135"
 			(at 170.688 85.09 90)
 			(show_name no)
@@
 			(project "8bit"
 				(path "/ce6ef060-f4bd-4228-ab8d-5cf6f386dba1/a913a341-ba12-46a1-b026-37d3a35c843c"
-					(reference "R115")
+					(reference "R135")
 					(unit 1)
 				)
@@
 		(in_pos_files yes)
 		(dnp no)
-		(property "Reference" "R113"
+		(property "Reference" "R133"
 			(at 160.528 85.09 90)
 			(show_name no)
@@
 			(project "8bit"
 				(path "/ce6ef060-f4bd-4228-ab8d-5cf6f386dba1/a913a341-ba12-46a1-b026-37d3a35c843c"
-					(reference "R113")
+					(reference "R133")
 					(unit 1)
 				)
@@
 		(in_pos_files yes)
 		(dnp no)
-		(property "Reference" "D94"
+		(property "Reference" "D95"
 			(at 145.288 90.17 0)
 			(show_name no)
@@
 			(project "8bit"
 				(path "/ce6ef060-f4bd-4228-ab8d-5cf6f386dba1/a913a341-ba12-46a1-b026-37d3a35c843c"
-					(reference "D94")
+					(reference "D95")
 					(unit 1)
 				)
@@
 		(in_pos_files yes)
 		(dnp no)
-		(property "Reference" "D96"
+		(property "Reference" "D97"
 			(at 155.448 90.17 0)
 			(show_name no)
@@
 			(project "8bit"
 				(path "/ce6ef060-f4bd-4228-ab8d-5cf6f386dba1/a913a341-ba12-46a1-b026-37d3a35c843c"
-					(reference "D96")
+					(reference "D97")
 					(unit 1)
 				)
@@
 		(in_pos_files yes)
 		(dnp no)
-		(property "Reference" "R116"
+		(property "Reference" "R136"
 			(at 175.768 85.09 90)
 			(show_name no)
@@
 			(project "8bit"
 				(path "/ce6ef060-f4bd-4228-ab8d-5cf6f386dba1/a913a341-ba12-46a1-b026-37d3a35c843c"
-					(reference "R116")
+					(reference "R136")
 					(unit 1)
 				)
@@
 		(in_pos_files yes)
 		(dnp no)
-		(property "Reference" "R110"
+		(property "Reference" "R130"
 			(at 145.288 85.09 90)
 			(show_name no)
@@
 			(project "8bit"
 				(path "/ce6ef060-f4bd-4228-ab8d-5cf6f386dba1/a913a341-ba12-46a1-b026-37d3a35c843c"
-					(reference "R110")
+					(reference "R130")
 					(unit 1)
 				)
@@
 		(in_pos_files yes)
 		(dnp no)
-		(property "Reference" "D95"
+		(property "Reference" "D96"
 			(at 150.368 90.17 0)
 			(show_name no)
@@
 			(project "8bit"
 				(path "/ce6ef060-f4bd-4228-ab8d-5cf6f386dba1/a913a341-ba12-46a1-b026-37d3a35c843c"
-					(reference "D95")
+					(reference "D96")
 					(unit 1)
 				)
@@
 		(in_pos_files yes)
 		(dnp no)
-		(property "Reference" "R112"
+		(property "Reference" "R132"
 			(at 155.448 85.09 90)
 			(show_name no)
@@
 			(project "8bit"
 				(path "/ce6ef060-f4bd-4228-ab8d-5cf6f386dba1/a913a341-ba12-46a1-b026-37d3a35c843c"
-					(reference "R112")
+					(reference "R132")
 					(unit 1)
 				)
@@
 		(dnp no)
 		(fields_autoplaced yes)
-		(property "Reference" "U71"
+		(property "Reference" "U38"
 			(at 72.3817 72.39 0)
 			(show_name no)
@@
 			(project "8bit"
 				(path "/ce6ef060-f4bd-4228-ab8d-5cf6f386dba1/a913a341-ba12-46a1-b026-37d3a35c843c"
-					(reference "U71")
+					(reference "U38")
 					(unit 1)
 				)
@@
 		(dnp no)
 		(fields_autoplaced yes)
-		(property "Reference" "#PWR076"
+		(property "Reference" "#PWR0118"
 			(at 205.74 97.79 0)
 			(hide yes)
@@
 			(project "8bit"
 				(path "/ce6ef060-f4bd-4228-ab8d-5cf6f386dba1/a913a341-ba12-46a1-b026-37d3a35c843c"
-					(reference "#PWR076")
+					(reference "#PWR0118")
 					(unit 1)
 				)
@@
 		(in_pos_files yes)
 		(dnp no)
-		(property "Reference" "R109"
+		(property "Reference" "R129"
 			(at 140.208 85.09 90)
 			(show_name no)
@@
 			(project "8bit"
 				(path "/ce6ef060-f4bd-4228-ab8d-5cf6f386dba1/a913a341-ba12-46a1-b026-37d3a35c843c"
-					(reference "R109")
+					(reference "R129")
 					(unit 1)
 				)
@@
 		(in_pos_files yes)
 		(dnp no)
-		(property "Reference" "D97"
+		(property "Reference" "D98"
 			(at 160.528 90.17 0)
 			(show_name no)
@@
 			(project "8bit"
 				(path "/ce6ef060-f4bd-4228-ab8d-5cf6f386dba1/a913a341-ba12-46a1-b026-37d3a35c843c"
-					(reference "D97")
+					(reference "D98")
 					(unit 1)
 				)
@@
 		(dnp no)
 		(fields_autoplaced yes)
-		(property "Reference" "#PWR0192"
+		(property "Reference" "#PWR0112"
 			(at 36.83 88.9 0)
 			(hide yes)
@@
 			(project "8bit"
 				(path "/ce6ef060-f4bd-4228-ab8d-5cf6f386dba1/a913a341-ba12-46a1-b026-37d3a35c843c"
-					(reference "#PWR0192")
+					(reference "#PWR0112")
 					(unit 1)
 				)
@@
 		(dnp no)
 		(fields_autoplaced yes)
-		(property "Reference" "U25"
+		(property "Reference" "U40"
 			(at 207.8833 50.8 0)
 			(show_name no)
@@
 			(project "8bit"
 				(path "/ce6ef060-f4bd-4228-ab8d-5cf6f386dba1/a913a341-ba12-46a1-b026-37d3a35c843c"
-					(reference "U25")
+					(reference "U40")
 					(unit 1)
 				)
@@
 		(in_pos_files yes)
 		(dnp no)
-		(property "Reference" "R114"
+		(property "Reference" "R134"
 			(at 165.608 85.09 90)
 			(show_name no)
@@
 			(project "8bit"
 				(path "/ce6ef060-f4bd-4228-ab8d-5cf6f386dba1/a913a341-ba12-46a1-b026-37d3a35c843c"
-					(reference "R114")
+					(reference "R134")
 					(unit 1)
 				)
@@
 		(in_pos_files yes)
 		(dnp no)
-		(property "Reference" "D93"
+		(property "Reference" "D94"
 			(at 140.208 90.17 0)
 			(show_name no)
@@
 			(project "8bit"
 				(path "/ce6ef060-f4bd-4228-ab8d-5cf6f386dba1/a913a341-ba12-46a1-b026-37d3a35c843c"
-					(reference "D93")
+					(reference "D94")
 					(unit 1)
 				)
@@
 		(in_pos_files yes)
 		(dnp no)
-		(property "Reference" "D100"
+		(property "Reference" "D101"
 			(at 175.768 90.17 0)
 			(show_name no)
@@
 			(project "8bit"
 				(path "/ce6ef060-f4bd-4228-ab8d-5cf6f386dba1/a913a341-ba12-46a1-b026-37d3a35c843c"
-					(reference "D100")
+					(reference "D101")
 					(unit 1)
 				)
@@
 		(in_pos_files yes)
 		(dnp no)
-		(property "Reference" "R111"
+		(property "Reference" "R131"
 			(at 150.368 85.09 90)
 			(show_name no)
@@
 			(project "8bit"
 				(path "/ce6ef060-f4bd-4228-ab8d-5cf6f386dba1/a913a341-ba12-46a1-b026-37d3a35c843c"
-					(reference "R111")
+					(reference "R131")
 					(unit 1)
 				)
@@
 		(in_pos_files yes)
 		(dnp no)
-		(property "Reference" "D99"
+		(property "Reference" "D100"
 			(at 170.688 90.17 0)
 			(show_name no)
@@
 			(project "8bit"
 				(path "/ce6ef060-f4bd-4228-ab8d-5cf6f386dba1/a913a341-ba12-46a1-b026-37d3a35c843c"
-					(reference "D99")
+					(reference "D100")
 					(unit 1)
 				)
@@
 		(in_pos_files yes)
 		(dnp no)
-		(property "Reference" "D98"
+		(property "Reference" "D99"
 			(at 165.608 90.17 0)
 			(show_name no)
@@
 			(project "8bit"
 				(path "/ce6ef060-f4bd-4228-ab8d-5cf6f386dba1/a913a341-ba12-46a1-b026-37d3a35c843c"
-					(reference "D98")
+					(reference "D99")
 					(unit 1)
 				)
@@
 		(dnp no)
 		(fields_autoplaced yes)
-		(property "Reference" "#PWR072"
+		(property "Reference" "#PWR0114"
 			(at 99.06 97.79 0)
 			(hide yes)
@@
 			(project "8bit"
 				(path "/ce6ef060-f4bd-4228-ab8d-5cf6f386dba1/a913a341-ba12-46a1-b026-37d3a35c843c"
-					(reference "#PWR072")
+					(reference "#PWR0114")
 					(unit 1)
 				)
@@
 		(in_pos_files yes)
 		(dnp no)
-		(property "Reference" "U71"
+		(property "Reference" "U38"
 			(at 44.704 68.326 0)
 			(show_name no)
@@
 			(project "8bit"
 				(path "/ce6ef060-f4bd-4228-ab8d-5cf6f386dba1/a913a341-ba12-46a1-b026-37d3a35c843c"
-					(reference "U71")
+					(reference "U38")
 					(unit 5)
 				)
@@
 		(in_pos_files yes)
 		(dnp no)
-		(property "Reference" "#PWR073"
+		(property "Reference" "#PWR0115"
 			(at 160.02 104.14 0)
 			(hide yes)
@@
 			(project "8bit"
 				(path "/ce6ef060-f4bd-4228-ab8d-5cf6f386dba1/a913a341-ba12-46a1-b026-37d3a35c843c"
-					(reference "#PWR073")
-					(unit 1)
-				)
+					(reference "#PWR0115")
+					(unit 1)
+				)
