File: schematic/register_b_c.kicad_sch (KiCad schematic)
At the start: 39 parts, among them U36 74LS573, U37 74LS245, U38 74LS573, U39 74LS245, U40 74LS245, U41 74LS245, U73 74LS08

Commit message: feat: address decoding completed, general clean up
Parts:
- renumbered D133 to D138, D141 to D139, D134 to D140, D142 to D141, D135 to D142, D136 to D144, D144 to D145, D137 to D146, D145 to D147, D138 to D148, D146 to D149, D139 to D150, D147 to D151, D140 to D152, D148 to D153, R149 to R173, R157 to R174, R150 to R175, R158 to R176, R151 to R177, R159 to R178, R152 to R179, R160 to R180, R153 to R181, R161 to R182, R154 to R183, R162 to R184, R155 to R185, R163 to R186, R156 to R187, R164 to R188, U73 to U63, U36 to U64, U38 to U65, U37 to U66, U39 to U67, U40 to U68, U41 to U69
