File: schematic/register_d_e.kicad_sch (KiCad schematic)
At the start: 39 parts, among them U42 74LS573, U43 74LS573, U44 74LS245, U45 74LS245, U46 74LS245, U47 74LS245, U74 74LS08

Commit message: feat: address decoding completed, general clean up
Parts:
- renumbered D149 to D154, D150 to D155, D151 to D156, D152 to D157, D153 to D158, D154 to D159, D155 to D160, D156 to D161, D157 to D162, D158 to D163, D159 to D164, D160 to D165, D161 to D166, D162 to D167, D163 to D168, D164 to D169, R165 to R189, R166 to R190, R167 to R191, R168 to R192, R169 to R193, R170 to R194, R171 to R195, R172 to R196, R173 to R197, R174 to R198, R175 to R199, R176 to R200, R177 to R201, R178 to R202, R179 to R203, R180 to R204, U74 to U70, U42 to U71, U43 to U72, U44 to U73, U45 to U74, U46 to U75, U47 to U76
