File: schematic/register_instruction.kicad_sch (KiCad schematic)
At the start: 20 parts, among them U54 74LS573, U75 74LS08, U98 ER_OLEDM0.91_1x-I2C

Commit message: feat: address decoding completed, general clean up
Parts:
- renumbered D101 to D170, D102 to D171, D103 to D172, D104 to D173, D105 to D174, D106 to D175, D107 to D176, D108 to D177, R117 to R205, R118 to R206, R119 to R207, R120 to R208, R121 to R209, R122 to R210, R123 to R211, R124 to R212, U75 to U50, U54 to U77, U98 to U78
Connections:
- no-connect marks 2 -> 16
