File: schematic/register_output.kicad_sch (KiCad schematic)
At the start: 15 parts, among them J2 EXTR, SW1 RST, U55 74LS573, U56 ATmega328-P, U57 D198K, U58 D198K, U59 D198K, U60 D198K, U76 74LS08

Commit message: feat: address decoding completed, general clean up
Parts:
- renumbered R202 to R213, R203 to R214, R197 to R215, R198 to R216, R199 to R217, R200 to R218, SW1 to SW4, U76 to U79, U55 to U80, U56 to U81, U57 to U82, U58 to U83, U59 to U84, U60 to U85
Changed lines of the file:
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@@
 		(in_pos_files yes)
 		(dnp no)
-		(property "Reference" "#PWR0159"
+		(property "Reference" "#PWR0226"
 			(at 144.78 92.71 0)
 			(hide yes)
@@
 			(project "8bit"
 				(path "/ce6ef060-f4bd-4228-ab8d-5cf6f386dba1/a46e9ff3-6e70-490d-91af-2a69eac568f7"
-					(reference "#PWR0159")
+					(reference "#PWR0226")
 					(unit 1)
 				)
@@
 		(in_pos_files yes)
 		(dnp no)
-		(property "Reference" "U60"
+		(property "Reference" "U85"
 			(at 200.66 127.508 0)
 			(show_name no)
@@
 			(project "8bit"
 				(path "/ce6ef060-f4bd-4228-ab8d-5cf6f386dba1/a46e9ff3-6e70-490d-91af-2a69eac568f7"
-					(reference "U60")
+					(reference "U85")
 					(unit 1)
 				)
@@
 		(dnp no)
 		(fields_autoplaced yes)
-		(property "Reference" "U76"
+		(property "Reference" "U79"
 			(at 52.0617 60.96 0)
 			(show_name no)
@@
 			(project "8bit"
 				(path "/ce6ef060-f4bd-4228-ab8d-5cf6f386dba1/a46e9ff3-6e70-490d-91af-2a69eac568f7"
-					(reference "U76")
+					(reference "U79")
 					(unit 1)
 				)
@@
 		(in_pos_files yes)
 		(dnp no)
-		(property "Reference" "R202"
+		(property "Reference" "R213"
 			(at 130.81 88.646 90)
 			(show_name no)
@@
 			(project "8bit"
 				(path "/ce6ef060-f4bd-4228-ab8d-5cf6f386dba1/a46e9ff3-6e70-490d-91af-2a69eac568f7"
-					(reference "R202")
+					(reference "R213")
 					(unit 1)
 				)
@@
 		(dnp no)
 		(fields_autoplaced yes)
-		(property "Reference" "#PWR0157"
+		(property "Reference" "#PWR0221"
 			(at 77.47 43.18 0)
 			(hide yes)
@@
 			(project "8bit"
 				(path "/ce6ef060-f4bd-4228-ab8d-5cf6f386dba1/a46e9ff3-6e70-490d-91af-2a69eac568f7"
-					(reference "#PWR0157")
+					(reference "#PWR0221")
 					(unit 1)
 				)
@@
 		(in_pos_files yes)
 		(dnp no)
-		(property "Reference" "U76"
+		(property "Reference" "U79"
 			(at 170.434 175.006 0)
 			(show_name no)
@@
 			(project "8bit"
 				(path "/ce6ef060-f4bd-4228-ab8d-5cf6f386dba1/a46e9ff3-6e70-490d-91af-2a69eac568f7"
-					(reference "U76")
+					(reference "U79")
 					(unit 5)
 				)
@@
 		(dnp no)
 		(fields_autoplaced yes)
-		(property "Reference" "#PWR0160"
+		(property "Reference" "#PWR0223"
 			(at 113.03 31.75 0)
 			(hide yes)
@@
 			(project "8bit"
 				(path "/ce6ef060-f4bd-4228-ab8d-5cf6f386dba1/a46e9ff3-6e70-490d-91af-2a69eac568f7"
-					(reference "#PWR0160")
+					(reference "#PWR0223")
 					(unit 1)
 				)
@@
 		(in_pos_files yes)
 		(dnp no)
-		(property "Reference" "R198"
+		(property "Reference" "R216"
 			(at 152.654 59.69 90)
 			(show_name no)
@@
 			(project "8bit"
 				(path "/ce6ef060-f4bd-4228-ab8d-5cf6f386dba1/a46e9ff3-6e70-490d-91af-2a69eac568f7"
-					(reference "R198")
+					(reference "R216")
 					(unit 1)
 				)
@@
 		(in_pos_files yes)
 		(dnp no)
-		(property "Reference" "U58"
+		(property "Reference" "U83"
 			(at 200.66 64.008 0)
 			(show_name no)
@@
 			(project "8bit"
 				(path "/ce6ef060-f4bd-4228-ab8d-5cf6f386dba1/a46e9ff3-6e70-490d-91af-2a69eac568f7"
-					(reference "U58")
+					(reference "U83")
 					(unit 1)
 				)
@@
 		(in_pos_files yes)
 		(dnp no)
-		(property "Reference" "#PWR0162"
+		(property "Reference" "#PWR0225"
 			(at 134.62 78.74 0)
 			(hide yes)
@@
 			(project "8bit"
 				(path "/ce6ef060-f4bd-4228-ab8d-5cf6f386dba1/a46e9ff3-6e70-490d-91af-2a69eac568f7"
-					(reference "#PWR0162")
+					(reference "#PWR0225")
 					(unit 1)
 				)
@@
 		(in_pos_files yes)
 		(dnp no)
-		(property "Reference" "R203"
+		(property "Reference" "R214"
 			(at 132.08 81.28 90)
 			(show_name no)
@@
 			(project "8bit"
 				(path "/ce6ef060-f4bd-4228-ab8d-5cf6f386dba1/a46e9ff3-6e70-490d-91af-2a69eac568f7"
-					(reference "R203")
+					(reference "R214")
 					(unit 1)
 				)
@@
 		(dnp no)
 		(fields_autoplaced yes)
-		(property "Reference" "U55"
+		(property "Reference" "U80"
 			(at 79.6133 39.37 0)
 			(show_name no)
@@
 			(project "8bit"
 				(path "/ce6ef060-f4bd-4228-ab8d-5cf6f386dba1/a46e9ff3-6e70-490d-91af-2a69eac568f7"
-					(reference "U55")
+					(reference "U80")
 					(unit 1)
 				)
@@
 		(in_pos_files yes)
 		(dnp no)
-		(property "Reference" "SW1"
+		(property "Reference" "SW4"
 			(at 139.7 80.518 0)
 			(show_name no)
@@
 			(project "8bit"
 				(path "/ce6ef060-f4bd-4228-ab8d-5cf6f386dba1/a46e9ff3-6e70-490d-91af-2a69eac568f7"
-					(reference "SW1")
+					(reference "SW4")
 					(unit 1)
 				)
@@
 		(in_pos_files yes)
 		(dnp no)
-		(property "Reference" "U59"
+		(property "Reference" "U84"
 			(at 200.914 95.25 0)
 			(show_name no)
@@
 			(project "8bit"
 				(path "/ce6ef060-f4bd-4228-ab8d-5cf6f386dba1/a46e9ff3-6e70-490d-91af-2a69eac568f7"
-					(reference "U59")
+					(reference "U84")
 					(unit 1)
 				)
@@
 		(dnp no)
 		(fields_autoplaced yes)
-		(property "Reference" "#PWR0202"
+		(property "Reference" "#PWR0228"
 			(at 162.56 195.58 0)
 			(hide yes)
@@
 			(project "8bit"
 				(path "/ce6ef060-f4bd-4228-ab8d-5cf6f386dba1/a46e9ff3-6e70-490d-91af-2a69eac568f7"
-					(reference "#PWR0202")
+					(reference "#PWR0228")
 					(unit 1)
 				)
@@
 		(dnp no)
 		(fields_autoplaced yes)
-		(property "Reference" "#PWR0201"
+		(property "Reference" "#PWR0227"
 			(at 162.56 167.64 0)
 			(hide yes)
@@
 			(project "8bit"
 				(path "/ce6ef060-f4bd-4228-ab8d-5cf6f386dba1/a46e9ff3-6e70-490d-91af-2a69eac568f7"
-					(reference "#PWR0201")
+					(reference "#PWR0227")
 					(unit 1)
 				)
@@
 		(dnp no)
 		(fields_autoplaced yes)
-		(property "Reference" "#PWR0158"
+		(property "Reference" "#PWR0222"
 			(at 77.47 86.36 0)
 			(hide yes)
@@
 			(project "8bit"
 				(path "/ce6ef060-f4bd-4228-ab8d-5cf6f386dba1/a46e9ff3-6e70-490d-91af-2a69eac568f7"
-					(reference "#PWR0158")
+					(reference "#PWR0222")
 					(unit 1)
 				)
@@
 		(dnp no)
 		(fields_autoplaced yes)
-		(property "Reference" "#PWR0161"
+		(property "Reference" "#PWR0224"
 			(at 113.03 87.63 0)
 			(hide yes)
@@
 			(project "8bit"
 				(path "/ce6ef060-f4bd-4228-ab8d-5cf6f386dba1/a46e9ff3-6e70-490d-91af-2a69eac568f7"
-					(reference "#PWR0161")
+					(reference "#PWR0224")
 					(unit 1)
 				)
@@
 		(in_pos_files yes)
 		(dnp no)
-		(property "Reference" "R200"
+		(property "Reference" "R218"
 			(at 152.654 64.77 90)
 			(show_name no)
@@
 			(project "8bit"
 				(path "/ce6ef060-f4bd-4228-ab8d-5cf6f386dba1/a46e9ff3-6e70-490d-91af-2a69eac568f7"
-					(reference "R200")
+					(reference "R218")
 					(unit 1)
 				)
@@
 		(in_pos_files yes)
 		(dnp no)
-		(property "Reference" "R197"
+		(property "Reference" "R215"
 			(at 152.654 57.15 90)
 			(show_name no)
@@
 			(project "8bit"
 				(path "/ce6ef060-f4bd-4228-ab8d-5cf6f386dba1/a46e9ff3-6e70-490d-91af-2a69eac568f7"
-					(reference "R197")
+					(reference "R215")
 					(unit 1)
 				)
@@
 		(in_pos_files yes)
 		(dnp no)
-		(property "Reference" "U57"
+		(property "Reference" "U82"
 			(at 200.66 31.75 0)
 			(show_name no)
@@
 			(project "8bit"
 				(path "/ce6ef060-f4bd-4228-ab8d-5cf6f386dba1/a46e9ff3-6e70-490d-91af-2a69eac568f7"
-					(reference "U57")
+					(reference "U82")
 					(unit 1)
 				)
@@
 		(in_pos_files yes)
 		(dnp no)
-		(property "Reference" "R199"
+		(property "Reference" "R217"
 			(at 152.654 62.23 90)
 			(show_name no)
@@
 			(project "8bit"
 				(path "/ce6ef060-f4bd-4228-ab8d-5cf6f386dba1/a46e9ff3-6e70-490d-91af-2a69eac568f7"
-					(reference "R199")
+					(reference "R217")
 					(unit 1)
 				)
@@
 		(in_pos_files yes)
 		(dnp no)
-		(property "Reference" "U56"
+		(property "Reference" "U81"
 			(at 102.362 25.654 0)
 			(show_name no)
@@
 			(project "8bit"
 				(path "/ce6ef060-f4bd-4228-ab8d-5cf6f386dba1/a46e9ff3-6e70-490d-91af-2a69eac568f7"
-					(reference "U56")
-					(unit 1)
-				)
+					(reference "U81")
+					(unit 1)
+				)
