File: schematic/register_temporary.kicad_sch (KiCad schematic)
At the start: 19 parts, among them U100 74LS573, U101 74LS245, U99 74LS08

Commit message: feat: address decoding completed, general clean up
Parts:
- renumbered D198 to D183, D199 to D184, D200 to D185, D201 to D186, D202 to D187, D203 to D188, D204 to D189, D205 to D190, R226 to R230, R227 to R231, R228 to R232, R229 to R233, R230 to R234, R231 to R235, R248 to R236, R249 to R237, U99 to U108, U100 to U109, U101 to U110
Changed lines of the file:
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@@
 		(dnp no)
 		(fields_autoplaced yes)
-		(property "Reference" "#PWR0271"
+		(property "Reference" "#PWR0282"
 			(at 55.88 72.39 0)
 			(hide yes)
@@
 			(project "8bit"
 				(path "/ce6ef060-f4bd-4228-ab8d-5cf6f386dba1/3f741fd1-4e21-4402-b927-a34a55bf0dfc"
-					(reference "#PWR0271")
+					(reference "#PWR0282")
 					(unit 1)
 				)
@@
 		(dnp no)
 		(fields_autoplaced yes)
-		(property "Reference" "#PWR0276"
+		(property "Reference" "#PWR0288"
 			(at 224.79 66.04 0)
 			(hide yes)
@@
 			(project "8bit"
 				(path "/ce6ef060-f4bd-4228-ab8d-5cf6f386dba1/3f741fd1-4e21-4402-b927-a34a55bf0dfc"
-					(reference "#PWR0276")
+					(reference "#PWR0288")
 					(unit 1)
 				)
@@
 		(in_pos_files yes)
 		(dnp no)
-		(property "Reference" "R228"
+		(property "Reference" "R232"
 			(at 169.418 96.52 90)
 			(show_name no)
@@
 			(project "8bit"
 				(path "/ce6ef060-f4bd-4228-ab8d-5cf6f386dba1/3f741fd1-4e21-4402-b927-a34a55bf0dfc"
-					(reference "R228")
+					(reference "R232")
 					(unit 1)
 				)
@@
 		(dnp no)
 		(fields_autoplaced yes)
-		(property "Reference" "U99"
+		(property "Reference" "U108"
 			(at 91.4317 83.82 0)
 			(show_name no)
@@
 			(project "8bit"
 				(path "/ce6ef060-f4bd-4228-ab8d-5cf6f386dba1/3f741fd1-4e21-4402-b927-a34a55bf0dfc"
-					(reference "U99")
+					(reference "U108")
 					(unit 1)
 				)
@@
 		(in_pos_files yes)
 		(dnp no)
-		(property "Reference" "R226"
+		(property "Reference" "R230"
 			(at 159.258 96.52 90)
 			(show_name no)
@@
 			(project "8bit"
 				(path "/ce6ef060-f4bd-4228-ab8d-5cf6f386dba1/3f741fd1-4e21-4402-b927-a34a55bf0dfc"
-					(reference "R226")
+					(reference "R230")
 					(unit 1)
 				)
@@
 		(in_pos_files yes)
 		(dnp no)
-		(property "Reference" "D198"
+		(property "Reference" "D183"
 			(at 159.258 101.6 0)
 			(show_name no)
@@
 			(project "8bit"
 				(path "/ce6ef060-f4bd-4228-ab8d-5cf6f386dba1/3f741fd1-4e21-4402-b927-a34a55bf0dfc"
-					(reference "D198")
+					(reference "D183")
 					(unit 1)
 				)
@@
 		(in_pos_files yes)
 		(dnp no)
-		(property "Reference" "D204"
+		(property "Reference" "D189"
 			(at 189.738 101.6 0)
 			(show_name no)
@@
 			(project "8bit"
 				(path "/ce6ef060-f4bd-4228-ab8d-5cf6f386dba1/3f741fd1-4e21-4402-b927-a34a55bf0dfc"
-					(reference "D204")
+					(reference "D189")
 					(unit 1)
 				)
@@
 		(dnp no)
 		(fields_autoplaced yes)
-		(property "Reference" "#PWR087"
+		(property "Reference" "#PWR0284"
 			(at 118.11 66.04 0)
 			(hide yes)
@@
 			(project "8bit"
 				(path "/ce6ef060-f4bd-4228-ab8d-5cf6f386dba1/3f741fd1-4e21-4402-b927-a34a55bf0dfc"
-					(reference "#PWR087")
+					(reference "#PWR0284")
 					(unit 1)
 				)
@@
 		(in_pos_files yes)
 		(dnp no)
-		(property "Reference" "#PWR0274"
+		(property "Reference" "#PWR0286"
 			(at 179.07 115.57 0)
 			(hide yes)
@@
 			(project "8bit"
 				(path "/ce6ef060-f4bd-4228-ab8d-5cf6f386dba1/3f741fd1-4e21-4402-b927-a34a55bf0dfc"
-					(reference "#PWR0274")
+					(reference "#PWR0286")
 					(unit 1)
 				)
@@
 		(in_pos_files yes)
 		(dnp no)
-		(property "Reference" "D200"
+		(property "Reference" "D185"
 			(at 169.418 101.6 0)
 			(show_name no)
@@
 			(project "8bit"
 				(path "/ce6ef060-f4bd-4228-ab8d-5cf6f386dba1/3f741fd1-4e21-4402-b927-a34a55bf0dfc"
-					(reference "D200")
+					(reference "D185")
 					(unit 1)
 				)
@@
 		(dnp no)
 		(fields_autoplaced yes)
-		(property "Reference" "#PWR0272"
+		(property "Reference" "#PWR0283"
 			(at 55.88 100.33 0)
 			(hide yes)
@@
 			(project "8bit"
 				(path "/ce6ef060-f4bd-4228-ab8d-5cf6f386dba1/3f741fd1-4e21-4402-b927-a34a55bf0dfc"
-					(reference "#PWR0272")
+					(reference "#PWR0283")
 					(unit 1)
 				)
@@
 		(in_pos_files yes)
 		(dnp no)
-		(property "Reference" "R231"
+		(property "Reference" "R235"
 			(at 184.658 96.52 90)
 			(show_name no)
@@
 			(project "8bit"
 				(path "/ce6ef060-f4bd-4228-ab8d-5cf6f386dba1/3f741fd1-4e21-4402-b927-a34a55bf0dfc"
-					(reference "R231")
+					(reference "R235")
 					(unit 1)
 				)
@@
 		(in_pos_files yes)
 		(dnp no)
-		(property "Reference" "U99"
+		(property "Reference" "U108"
 			(at 63.754 79.756 0)
 			(show_name no)
@@
 			(project "8bit"
 				(path "/ce6ef060-f4bd-4228-ab8d-5cf6f386dba1/3f741fd1-4e21-4402-b927-a34a55bf0dfc"
-					(reference "U99")
+					(reference "U108")
 					(unit 5)
 				)
@@
 		(in_pos_files yes)
 		(dnp no)
-		(property "Reference" "R230"
+		(property "Reference" "R234"
 			(at 179.578 96.52 90)
 			(show_name no)
@@
 			(project "8bit"
 				(path "/ce6ef060-f4bd-4228-ab8d-5cf6f386dba1/3f741fd1-4e21-4402-b927-a34a55bf0dfc"
-					(reference "R230")
+					(reference "R234")
 					(unit 1)
 				)
@@
 		(in_pos_files yes)
 		(dnp no)
-		(property "Reference" "D199"
+		(property "Reference" "D184"
 			(at 164.338 101.6 0)
 			(show_name no)
@@
 			(project "8bit"
 				(path "/ce6ef060-f4bd-4228-ab8d-5cf6f386dba1/3f741fd1-4e21-4402-b927-a34a55bf0dfc"
-					(reference "D199")
+					(reference "D184")
 					(unit 1)
 				)
@@
 		(in_pos_files yes)
 		(dnp no)
-		(property "Reference" "R248"
+		(property "Reference" "R236"
 			(at 189.738 96.52 90)
 			(show_name no)
@@
 			(project "8bit"
 				(path "/ce6ef060-f4bd-4228-ab8d-5cf6f386dba1/3f741fd1-4e21-4402-b927-a34a55bf0dfc"
-					(reference "R248")
+					(reference "R236")
 					(unit 1)
 				)
@@
 		(dnp no)
 		(fields_autoplaced yes)
-		(property "Reference" "#PWR0273"
+		(property "Reference" "#PWR0285"
 			(at 118.11 109.22 0)
 			(hide yes)
@@
 			(project "8bit"
 				(path "/ce6ef060-f4bd-4228-ab8d-5cf6f386dba1/3f741fd1-4e21-4402-b927-a34a55bf0dfc"
-					(reference "#PWR0273")
+					(reference "#PWR0285")
 					(unit 1)
 				)
@@
 		(dnp no)
 		(fields_autoplaced yes)
-		(property "Reference" "#PWR0277"
+		(property "Reference" "#PWR0289"
 			(at 224.79 109.22 0)
 			(hide yes)
@@
 			(project "8bit"
 				(path "/ce6ef060-f4bd-4228-ab8d-5cf6f386dba1/3f741fd1-4e21-4402-b927-a34a55bf0dfc"
-					(reference "#PWR0277")
+					(reference "#PWR0289")
 					(unit 1)
 				)
@@
 		(in_pos_files yes)
 		(dnp no)
-		(property "Reference" "R249"
+		(property "Reference" "R237"
 			(at 194.818 96.52 90)
 			(show_name no)
@@
 			(project "8bit"
 				(path "/ce6ef060-f4bd-4228-ab8d-5cf6f386dba1/3f741fd1-4e21-4402-b927-a34a55bf0dfc"
-					(reference "R249")
+					(reference "R237")
 					(unit 1)
 				)
@@
 		(in_pos_files yes)
 		(dnp no)
-		(property "Reference" "D202"
+		(property "Reference" "D187"
 			(at 179.578 101.6 0)
 			(show_name no)
@@
 			(project "8bit"
 				(path "/ce6ef060-f4bd-4228-ab8d-5cf6f386dba1/3f741fd1-4e21-4402-b927-a34a55bf0dfc"
-					(reference "D202")
+					(reference "D187")
 					(unit 1)
 				)
@@
 		(in_pos_files yes)
 		(dnp no)
-		(property "Reference" "D205"
+		(property "Reference" "D190"
 			(at 194.818 101.6 0)
 			(show_name no)
@@
 			(project "8bit"
 				(path "/ce6ef060-f4bd-4228-ab8d-5cf6f386dba1/3f741fd1-4e21-4402-b927-a34a55bf0dfc"
-					(reference "D205")
+					(reference "D190")
 					(unit 1)
 				)
@@
 		(in_pos_files yes)
 		(dnp no)
-		(property "Reference" "D201"
+		(property "Reference" "D186"
 			(at 174.498 101.6 0)
 			(show_name no)
@@
 			(project "8bit"
 				(path "/ce6ef060-f4bd-4228-ab8d-5cf6f386dba1/3f741fd1-4e21-4402-b927-a34a55bf0dfc"
-					(reference "D201")
+					(reference "D186")
 					(unit 1)
 				)
@@
 		(in_pos_files yes)
 		(dnp no)
-		(property "Reference" "#PWR0275"
+		(property "Reference" "#PWR0287"
 			(at 207.01 96.52 0)
 			(hide yes)
@@
 			(project "8bit"
 				(path "/ce6ef060-f4bd-4228-ab8d-5cf6f386dba1/3f741fd1-4e21-4402-b927-a34a55bf0dfc"
-					(reference "#PWR0275")
+					(reference "#PWR0287")
 					(unit 1)
 				)
@@
 		(dnp no)
 		(fields_autoplaced yes)
-		(property "Reference" "U100"
+		(property "Reference" "U109"
 			(at 120.2533 62.23 0)
 			(show_name no)
@@
 			(project "8bit"
 				(path "/ce6ef060-f4bd-4228-ab8d-5cf6f386dba1/3f741fd1-4e21-4402-b927-a34a55bf0dfc"
-					(reference "U100")
+					(reference "U109")
 					(unit 1)
 				)
@@
 		(in_pos_files yes)
 		(dnp no)
-		(property "Reference" "R229"
+		(property "Reference" "R233"
 			(at 174.498 96.52 90)
 			(show_name no)
@@
 			(project "8bit"
 				(path "/ce6ef060-f4bd-4228-ab8d-5cf6f386dba1/3f741fd1-4e21-4402-b927-a34a55bf0dfc"
-					(reference "R229")
+					(reference "R233")
 					(unit 1)
 				)
@@
 		(in_pos_files yes)
 		(dnp no)
-		(property "Reference" "D203"
+		(property "Reference" "D188"
 			(at 184.658 101.6 0)
 			(show_name no)
@@
 			(project "8bit"
 				(path "/ce6ef060-f4bd-4228-ab8d-5cf6f386dba1/3f741fd1-4e21-4402-b927-a34a55bf0dfc"
-					(reference "D203")
+					(reference "D188")
 					(unit 1)
 				)
@@
 		(dnp no)
 		(fields_autoplaced yes)
-		(property "Reference" "U101"
+		(property "Reference" "U110"
 			(at 226.9333 62.23 0)
 			(show_name no)
@@
 			(project "8bit"
 				(path "/ce6ef060-f4bd-4228-ab8d-5cf6f386dba1/3f741fd1-4e21-4402-b927-a34a55bf0dfc"
-					(reference "U101")
+					(reference "U110")
 					(unit 1)
 				)
@@
 		(in_pos_files yes)
 		(dnp no)
-		(property "Reference" "R227"
+		(property "Reference" "R231"
 			(at 164.338 96.52 90)
 			(show_name no)
@@
 			(project "8bit"
 				(path "/ce6ef060-f4bd-4228-ab8d-5cf6f386dba1/3f741fd1-4e21-4402-b927-a34a55bf0dfc"
-					(reference "R227")
-					(unit 1)
-				)
+					(reference "R231")
+					(unit 1)
+				)
