File: schematic/rom.kicad_sch (KiCad schematic)
At the start: 18 parts, among them U21 74LS245, U22 KM28C64A

Commit message: feat: address decoding completed, general clean up
Parts:
- renumbered D57 to D77, D58 to D78, D59 to D79, D60 to D80, D61 to D81, D62 to D82, D63 to D83, D64 to D84, R57 to R110, R58 to R111, R59 to R112, R60 to R113, R61 to R114, R62 to R115, R63 to R116, R64 to R117, U22 to U35, U21 to U36
Changed lines of the file:
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@@
 		(dnp no)
 		(fields_autoplaced yes)
-		(property "Reference" "#PWR059"
+		(property "Reference" "#PWR0100"
 			(at 181.61 115.57 0)
 			(hide yes)
@@
 			(project "8bit"
 				(path "/ce6ef060-f4bd-4228-ab8d-5cf6f386dba1/261ad9ec-e380-49c1-b1fc-50080f75aeb8"
-					(reference "#PWR059")
+					(reference "#PWR0100")
 					(unit 1)
 				)
@@
 		(in_pos_files yes)
 		(dnp no)
-		(property "Reference" "R60"
+		(property "Reference" "R113"
 			(at 131.318 109.22 90)
 			(show_name no)
@@
 			(project "8bit"
 				(path "/ce6ef060-f4bd-4228-ab8d-5cf6f386dba1/261ad9ec-e380-49c1-b1fc-50080f75aeb8"
-					(reference "R60")
+					(reference "R113")
 					(unit 1)
 				)
@@
 		(dnp no)
 		(fields_autoplaced yes)
-		(property "Reference" "#PWR058"
+		(property "Reference" "#PWR096"
 			(at 101.6 133.35 0)
 			(hide yes)
@@
 			(project "8bit"
 				(path "/ce6ef060-f4bd-4228-ab8d-5cf6f386dba1/261ad9ec-e380-49c1-b1fc-50080f75aeb8"
-					(reference "#PWR058")
+					(reference "#PWR096")
 					(unit 1)
 				)
@@
 		(in_pos_files yes)
 		(dnp no)
-		(property "Reference" "D58"
+		(property "Reference" "D78"
 			(at 121.158 114.3 0)
 			(show_name no)
@@
 			(project "8bit"
 				(path "/ce6ef060-f4bd-4228-ab8d-5cf6f386dba1/261ad9ec-e380-49c1-b1fc-50080f75aeb8"
-					(reference "D58")
+					(reference "D78")
 					(unit 1)
 				)
@@
 		(in_pos_files yes)
 		(dnp no)
-		(property "Reference" "D64"
+		(property "Reference" "D84"
 			(at 151.638 114.3 0)
 			(show_name no)
@@
 			(project "8bit"
 				(path "/ce6ef060-f4bd-4228-ab8d-5cf6f386dba1/261ad9ec-e380-49c1-b1fc-50080f75aeb8"
-					(reference "D64")
+					(reference "D84")
 					(unit 1)
 				)
@@
 		(dnp no)
 		(fields_autoplaced yes)
-		(property "Reference" "#PWR061"
+		(property "Reference" "#PWR094"
 			(at 88.9 119.38 0)
 			(hide yes)
@@
 			(project "8bit"
 				(path "/ce6ef060-f4bd-4228-ab8d-5cf6f386dba1/261ad9ec-e380-49c1-b1fc-50080f75aeb8"
-					(reference "#PWR061")
+					(reference "#PWR094")
 					(unit 1)
 				)
@@
 		(in_pos_files yes)
 		(dnp no)
-		(property "Reference" "D61"
+		(property "Reference" "D81"
 			(at 136.398 114.3 0)
 			(show_name no)
@@
 			(project "8bit"
 				(path "/ce6ef060-f4bd-4228-ab8d-5cf6f386dba1/261ad9ec-e380-49c1-b1fc-50080f75aeb8"
-					(reference "D61")
+					(reference "D81")
 					(unit 1)
 				)
@@
 		(in_pos_files yes)
 		(dnp no)
-		(property "Reference" "D59"
+		(property "Reference" "D79"
 			(at 126.238 114.3 0)
 			(show_name no)
@@
 			(project "8bit"
 				(path "/ce6ef060-f4bd-4228-ab8d-5cf6f386dba1/261ad9ec-e380-49c1-b1fc-50080f75aeb8"
-					(reference "D59")
+					(reference "D79")
 					(unit 1)
 				)
@@
 		(in_pos_files yes)
 		(dnp no)
-		(property "Reference" "R58"
+		(property "Reference" "R111"
 			(at 121.158 109.22 90)
 			(show_name no)
@@
 			(project "8bit"
 				(path "/ce6ef060-f4bd-4228-ab8d-5cf6f386dba1/261ad9ec-e380-49c1-b1fc-50080f75aeb8"
-					(reference "R58")
+					(reference "R111")
 					(unit 1)
 				)
@@
 		(in_pos_files yes)
 		(dnp no)
-		(property "Reference" "D60"
+		(property "Reference" "D80"
 			(at 131.318 114.3 0)
 			(show_name no)
@@
 			(project "8bit"
 				(path "/ce6ef060-f4bd-4228-ab8d-5cf6f386dba1/261ad9ec-e380-49c1-b1fc-50080f75aeb8"
-					(reference "D60")
+					(reference "D80")
 					(unit 1)
 				)
@@
 		(in_pos_files yes)
 		(dnp no)
-		(property "Reference" "R63"
+		(property "Reference" "R116"
 			(at 146.558 109.22 90)
 			(show_name no)
@@
 			(project "8bit"
 				(path "/ce6ef060-f4bd-4228-ab8d-5cf6f386dba1/261ad9ec-e380-49c1-b1fc-50080f75aeb8"
-					(reference "R63")
+					(reference "R116")
 					(unit 1)
 				)
@@
 		(in_pos_files yes)
 		(dnp no)
-		(property "Reference" "R57"
+		(property "Reference" "R110"
 			(at 116.078 109.22 90)
 			(show_name no)
@@
 			(project "8bit"
 				(path "/ce6ef060-f4bd-4228-ab8d-5cf6f386dba1/261ad9ec-e380-49c1-b1fc-50080f75aeb8"
-					(reference "R57")
+					(reference "R110")
 					(unit 1)
 				)
@@
 		(in_pos_files yes)
 		(dnp no)
-		(property "Reference" "#PWR060"
+		(property "Reference" "#PWR098"
 			(at 163.83 102.87 0)
 			(hide yes)
@@
 			(project "8bit"
 				(path "/ce6ef060-f4bd-4228-ab8d-5cf6f386dba1/261ad9ec-e380-49c1-b1fc-50080f75aeb8"
-					(reference "#PWR060")
+					(reference "#PWR098")
 					(unit 1)
 				)
@@
 		(dnp no)
 		(fields_autoplaced yes)
-		(property "Reference" "#PWR054"
+		(property "Reference" "#PWR095"
 			(at 101.6 74.93 0)
 			(hide yes)
@@
 			(project "8bit"
 				(path "/ce6ef060-f4bd-4228-ab8d-5cf6f386dba1/261ad9ec-e380-49c1-b1fc-50080f75aeb8"
-					(reference "#PWR054")
+					(reference "#PWR095")
 					(unit 1)
 				)
@@
 		(in_pos_files yes)
 		(dnp no)
-		(property "Reference" "R59"
+		(property "Reference" "R112"
 			(at 126.238 109.22 90)
 			(show_name no)
@@
 			(project "8bit"
 				(path "/ce6ef060-f4bd-4228-ab8d-5cf6f386dba1/261ad9ec-e380-49c1-b1fc-50080f75aeb8"
-					(reference "R59")
+					(reference "R112")
 					(unit 1)
 				)
@@
 		(in_pos_files yes)
 		(dnp no)
-		(property "Reference" "D62"
+		(property "Reference" "D82"
 			(at 141.478 114.3 0)
 			(show_name no)
@@
 			(project "8bit"
 				(path "/ce6ef060-f4bd-4228-ab8d-5cf6f386dba1/261ad9ec-e380-49c1-b1fc-50080f75aeb8"
-					(reference "D62")
+					(reference "D82")
 					(unit 1)
 				)
@@
 		(in_pos_files yes)
 		(dnp no)
-		(property "Reference" "R62"
+		(property "Reference" "R115"
 			(at 141.478 109.22 90)
 			(show_name no)
@@
 			(project "8bit"
 				(path "/ce6ef060-f4bd-4228-ab8d-5cf6f386dba1/261ad9ec-e380-49c1-b1fc-50080f75aeb8"
-					(reference "R62")
+					(reference "R115")
 					(unit 1)
 				)
@@
 		(dnp no)
 		(fields_autoplaced yes)
-		(property "Reference" "U22"
+		(property "Reference" "U35"
 			(at 103.7433 68.58 0)
 			(show_name no)
@@
 			(project "8bit"
 				(path "/ce6ef060-f4bd-4228-ab8d-5cf6f386dba1/261ad9ec-e380-49c1-b1fc-50080f75aeb8"
-					(reference "U22")
+					(reference "U35")
 					(unit 1)
 				)
@@
 		(in_pos_files yes)
 		(dnp no)
-		(property "Reference" "R64"
+		(property "Reference" "R117"
 			(at 151.638 109.22 90)
 			(show_name no)
@@
 			(project "8bit"
 				(path "/ce6ef060-f4bd-4228-ab8d-5cf6f386dba1/261ad9ec-e380-49c1-b1fc-50080f75aeb8"
-					(reference "R64")
+					(reference "R117")
 					(unit 1)
 				)
@@
 		(in_pos_files yes)
 		(dnp no)
-		(property "Reference" "R61"
+		(property "Reference" "R114"
 			(at 136.398 109.22 90)
 			(show_name no)
@@
 			(project "8bit"
 				(path "/ce6ef060-f4bd-4228-ab8d-5cf6f386dba1/261ad9ec-e380-49c1-b1fc-50080f75aeb8"
-					(reference "R61")
+					(reference "R114")
 					(unit 1)
 				)
@@
 		(in_pos_files yes)
 		(dnp no)
-		(property "Reference" "D63"
+		(property "Reference" "D83"
 			(at 146.558 114.3 0)
 			(show_name no)
@@
 			(project "8bit"
 				(path "/ce6ef060-f4bd-4228-ab8d-5cf6f386dba1/261ad9ec-e380-49c1-b1fc-50080f75aeb8"
-					(reference "D63")
+					(reference "D83")
 					(unit 1)
 				)
@@
 		(in_pos_files yes)
 		(dnp no)
-		(property "Reference" "#PWR056"
+		(property "Reference" "#PWR097"
 			(at 135.89 128.27 0)
 			(hide yes)
@@
 			(project "8bit"
 				(path "/ce6ef060-f4bd-4228-ab8d-5cf6f386dba1/261ad9ec-e380-49c1-b1fc-50080f75aeb8"
-					(reference "#PWR056")
+					(reference "#PWR097")
 					(unit 1)
 				)
@@
 		(dnp no)
 		(fields_autoplaced yes)
-		(property "Reference" "#PWR057"
+		(property "Reference" "#PWR099"
 			(at 181.61 72.39 0)
 			(hide yes)
@@
 			(project "8bit"
 				(path "/ce6ef060-f4bd-4228-ab8d-5cf6f386dba1/261ad9ec-e380-49c1-b1fc-50080f75aeb8"
-					(reference "#PWR057")
+					(reference "#PWR099")
 					(unit 1)
 				)
@@
 		(dnp no)
 		(fields_autoplaced yes)
-		(property "Reference" "U21"
+		(property "Reference" "U36"
 			(at 183.7533 68.58 0)
 			(show_name no)
@@
 			(project "8bit"
 				(path "/ce6ef060-f4bd-4228-ab8d-5cf6f386dba1/261ad9ec-e380-49c1-b1fc-50080f75aeb8"
-					(reference "U21")
+					(reference "U36")
 					(unit 1)
 				)
@@
 		(in_pos_files yes)
 		(dnp no)
-		(property "Reference" "D57"
+		(property "Reference" "D77"
 			(at 116.078 114.3 0)
 			(show_name no)
@@
 			(project "8bit"
 				(path "/ce6ef060-f4bd-4228-ab8d-5cf6f386dba1/261ad9ec-e380-49c1-b1fc-50080f75aeb8"
-					(reference "D57")
-					(unit 1)
-				)
+					(reference "D77")
+					(unit 1)
+				)
