File: schematic/alu.kicad_sch (KiCad schematic)
At the start: 53 parts, among them U28 74LS181, U29 74LS181, U30 74LS245, U31 74LS245, U32 74LS573, U33 74LS08, U34 74LS02, U35 74LS04, U72 74LS08, U75 74LS08, U77 74LS86, U96 74LS573, U97 74LS157

Commit message: feat: address decoding completed, general clean up
Parts:
- added unit 5 of U57
- renumbered D117 to D118, D118 to D119, D119 to D120, D120 to D121, D121 to D122, D122 to D123, D123 to D124, D124 to D125, D109 to D126, D110 to D127, D111 to D128, D112 to D129, D113 to D130, D114 to D131, D115 to D132, D116 to D133, D129 to D134, D130 to D135, D131 to D136, D132 to D137, R133 to R153, R134 to R154, R135 to R155, R136 to R156, R137 to R157, R138 to R158, R139 to R159, R140 to R160, R125 to R161, R126 to R162, R127 to R163, R128 to R164, R129 to R165, R130 to R166, R131 to R167, R132 to R168, R145 to R169, R146 to R170, R147 to R171, R148 to R172, U75 to U50, U34 to U51, U72 to U52, U35 to U53, U96 to U54, U31 to U55, U77 to U56, U33 to U57, U28 to U58, U29 to U59, U97 to U60, U32 to U61, U30 to U62
Connections:
- net +5V: now also U57.14 (VCC)
- net GND: now also U57.7 (GND)

Commit message: chore: update bom and footprintss
Parts:
- U54: footprint (none) -> Package_DIP:DIP-20_W7.62mm_Socket
- U60: footprint (none) -> Package_DIP:DIP-16_W7.62mm_Socket
Changed lines of the file:
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@@
 			)
 		)
-		(property "Footprint" ""
+		(property "Footprint" "Package_DIP:DIP-16_W7.62mm_Socket"
 			(at 278.13 210.82 0)
 			(hide yes)
@@
 			)
 		)
-		(property "Footprint" ""
+		(property "Footprint" "Package_DIP:DIP-20_W7.62mm_Socket"
 			(at 58.42 102.87 0)
 			(hide yes)
