File: schematic/cf_reader.kicad_sch (KiCad schematic)
At the start: 21 parts, among them J1 CF, U23 74LS245

Commit message: feat: address decoding completed, general clean up
Parts:
- added R118, R119: 1k, symbol Device:R
- renumbered D84 to D85, D85 to D86, D86 to D87, D87 to D88, D88 to D89, D89 to D90, D90 to D91, D91 to D92, D92 to D93, R68 to R120, R101 to R121, R102 to R122, R103 to R123, R104 to R124, R105 to R125, R106 to R126, R107 to R127, R108 to R128, U23 to U37
Connections:
- net +5V: now also R118.2, R119.2
- net ~{CF_RD}: now also R119.1
- net ~{CF_WR}: now also R118.1

Commit message: chore: update bom and footprintss
Parts:
- R118, R119: footprint (none) -> Resistor_SMD:R_0805_2012Metric
Other:
- moved on the sheet: D85, D86, D87, D88, D89, D90, D91, D92, D93, J1, JP1, R118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
