File: schematic/instruction_decoder.kicad_sch (KiCad schematic)
At the start: 4 parts, among them U63 27C512, U64 27C512, U65 27C512, U66 27C512

Commit message: feat: address decoding completed, general clean up
Parts:
- added U93, U94, U95, U96: 74LS04, symbol easyeda2kicad:74LS04
- added U97, U98, U99: 74LS154, symbol 74xx:74LS154
- renumbered U63 to U89, U64 to U90, U65 to U91, U66 to U92
Connections:
- net +5V: now also U93.14 (VCC), U94.14 (VCC), U95.14 (VCC), U96.14 (VCC), U97.24 (VCC), U98.24 (VCC), U99.24 (VCC)
- net GND: now also U93.7 (GND), U94.7 (GND), U95.7 (GND), U96.7 (GND), U97.12 (GND), U97.18 (E0), U97.19 (E1), U98.12 (GND), U98.18 (E0), U98.19 (E1), U99.12 (GND), U99.18 (E0), U99.19 (E1), U99.20 (A3)
- net PC_E: now reaches U92.11 (D0)
- net SC_RST: now reaches U92.12 (D1)
- net RAM_I: now reaches U92.13 (D2)
- net ALU_CARRY: now reaches U92.15 (D3)
- net MAR_INC: now reaches U92.16 (D4)
- net LCD_I: now reaches U92.17 (D5)
- net ALU_S0: now reaches U91.11 (D0)
- net ALU_S1: now reaches U91.12 (D1)
- net ALU_S2: now reaches U91.13 (D2)
- net ALU_S3: now reaches U91.15 (D3)
- net ALU_M: now reaches U91.16 (D4)
- net FR_I: now reaches U91.17 (D5)
- net at U91.18 (D6): now also U94.9
- net at U91.19 (D7): now also U94.11
- net HLT: now reaches U89.11 (D0)
- net OUT_MUX1: now reaches U89.12 (D1)
- net OUT_MUX1: now also U97.23 (A0)
- net OUT_MUX2: now reaches U89.13 (D2)
- net OUT_MUX2: now also U97.22 (A1)
- net OUT_MUX3: now reaches U89.15 (D3)
- net OUT_MUX3: now also U97.21 (A2)
- net OUT_MUX4: now reaches U89.16 (D4)
- net OUT_MUX4: now also U97.20 (A3)
- net ADDR_MUX1: now reaches U89.17 (D5)
- net ADDR_MUX1: now also U99.23 (A0)
- net ADDR_MUX2: now reaches U89.18 (D6)
- net ADDR_MUX2: now also U99.22 (A1)
- net ADDR_MUX3: now reaches U89.19 (D7)
- net ADDR_MUX3: now also U99.21 (A2)
- net IN_MUX1: now reaches U90.11 (D0)
- net IN_MUX1: now also U98.23 (A0)
- net IN_MUX2: now reaches U90.12 (D1)
- net IN_MUX2: now also U98.22 (A1)
- net IN_MUX3: now reaches U90.13 (D2)
- net IN_MUX3: now also U98.21 (A2)
- net IN_MUX4: now reaches U90.15 (D3)
- net IN_MUX4: now also U98.20 (A3)
- net at U90.16 (D4): now also U93.13
- net at U90.17 (D5): now also U94.1
- net at U90.18 (D6): now also U94.3
- net at U90.19 (D7): now also U94.5
- new net: U96.11, U98.10 (S9)
- new net: U95.13, U98.5 (S4)
- new net: U95.11, U98.4 (S3)
- new net: U96.13, U98.11 (S10)
- new net: U93.1, U98.13 (S11)
- new net: U93.3, U98.14 (S12)
- new net: U93.5, U98.15 (S13)
- new net: U93.9, U98.16 (S14)
- new net: U93.11, U98.17 (S15)
- new net: U95.5, U98.2 (S1)
- new net: U95.9, U98.3 (S2)
- new net: U96.1, U98.6 (S5)
- new net: U96.3, U98.7 (S6)
- new net: U96.5, U98.8 (S7)
- new net: U96.9, U98.9 (S8)
- new net: U95.1, U97.9 (S8)
- new net ALU_B_I: U93.10
- new net IR_I: U93.4
- new net MAR_H_I: U96.10
- new net MAR_L_I: U96.8
- new net OUTPUT_I: U93.8
- new net RAM_O: U95.2
- new net REG_A_I: U95.6
- new net REG_B_I: U95.8
- new net REG_C_I: U95.10
- new net REG_D_I: U95.12
- new net REG_E_I: U96.2
- new net REG_H_I: U96.6
- new net REG_L_I: U96.4
- new net REG_T_I: U93.6
- new net SP_H_I: U93.2
- new net SP_L_I: U96.12
- new net ~{ALU_O}: U97.10 (S9)
- new net ~{DEC_H}: U94.2
- new net ~{INC_H}: U93.12
- new net ~{JMP_H}: U94.10
- new net ~{JMP_L}: U94.8
- new net ~{MAR_O}: U99.7 (S6)
- new net ~{PAIR_BC_O}: U99.2 (S1)
- new net ~{PAIR_DE_O}: U99.3 (S2)
- new net ~{PAIR_HL_O}: U99.4 (S3)
- new net ~{PC_B_HOUT}: U97.16 (S14)
- new net ~{PC_B_LOUT}: U97.15 (S13)
- new net ~{PC_O}: U99.6 (S5)
- new net ~{POP}: U94.4
- new net ~{PUSH}: U94.6
- new net ~{RAR_OUT}: U97.14 (S12)
- new net ~{REG_A_O}: U97.2 (S1)
- new net ~{REG_B_O}: U97.3 (S2)
- new net ~{REG_C_O}: U97.4 (S3)
- new net ~{REG_D_O}: U97.5 (S4)
- new net ~{REG_E_O}: U97.6 (S5)
- new net ~{REG_H_O}: U97.8 (S7)
- new net ~{REG_L_O}: U97.7 (S6)
- new net ~{REG_T_O}: U97.11 (S10)
- new net ~{RRC_OUT}: U97.13 (S11)
- new net ~{SP_O}: U99.5 (S4)
- no-connect marks 0 -> 15
Other:
- note added: "ALL 74LS04"

Commit message: chore: update bom and footprintss
Parts:
- U93, U94, U95, U96: footprint (none) -> Package_DIP:DIP-14_W7.62mm_Socket
- U97, U98, U99: footprint (none) -> Package_DIP:DIP-24_W15.24mm_Socket
Changed lines of the file:
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@@
 			)
 		)
-		(property "Footprint" ""
+		(property "Footprint" "Package_DIP:DIP-14_W7.62mm_Socket"
 			(at 200.66 124.46 0)
 			(hide yes)
@@
 			)
 		)
-		(property "Footprint" ""
+		(property "Footprint" "Package_DIP:DIP-14_W7.62mm_Socket"
 			(at 200.66 111.76 0)
 			(hide yes)
@@
 			)
 		)
-		(property "Footprint" ""
+		(property "Footprint" "Package_DIP:DIP-14_W7.62mm_Socket"
 			(at 200.66 109.22 0)
 			(hide yes)
@@
 			)
 		)
-		(property "Footprint" ""
+		(property "Footprint" "Package_DIP:DIP-14_W7.62mm_Socket"
 			(at 99.06 173.99 0)
 			(hide yes)
@@
 			)
 		)
-		(property "Footprint" ""
+		(property "Footprint" "Package_DIP:DIP-14_W7.62mm_Socket"
 			(at 222.25 255.27 0)
 			(hide yes)
@@
 			)
 		)
-		(property "Footprint" ""
+		(property "Footprint" "Package_DIP:DIP-24_W15.24mm_Socket"
 			(at 179.07 119.38 0)
 			(hide yes)
@@
 			)
 		)
-		(property "Footprint" ""
+		(property "Footprint" "Package_DIP:DIP-14_W7.62mm_Socket"
 			(at 99.06 100.33 0)
 			(hide yes)
@@
 			)
 		)
-		(property "Footprint" ""
+		(property "Footprint" "Package_DIP:DIP-14_W7.62mm_Socket"
 			(at 200.66 114.3 0)
 			(hide yes)
@@
 			)
 		)
-		(property "Footprint" ""
+		(property "Footprint" "Package_DIP:DIP-14_W7.62mm_Socket"
 			(at 99.06 105.41 0)
 			(hide yes)
@@
 			)
 		)
-		(property "Footprint" ""
+		(property "Footprint" "Package_DIP:DIP-14_W7.62mm_Socket"
 			(at 99.06 97.79 0)
 			(hide yes)
@@
 			)
 		)
-		(property "Footprint" ""
+		(property "Footprint" "Package_DIP:DIP-24_W15.24mm_Socket"
 			(at 179.07 186.69 0)
 			(hide yes)
@@
 			)
 		)
-		(property "Footprint" ""
+		(property "Footprint" "Package_DIP:DIP-14_W7.62mm_Socket"
 			(at 200.66 119.38 0)
 			(hide yes)
@@
 			)
 		)
-		(property "Footprint" ""
+		(property "Footprint" "Package_DIP:DIP-14_W7.62mm_Socket"
 			(at 200.66 116.84 0)
 			(hide yes)
@@
 			)
 		)
-		(property "Footprint" ""
+		(property "Footprint" "Package_DIP:DIP-14_W7.62mm_Socket"
 			(at 200.66 137.16 0)
 			(hide yes)
@@
 			)
 		)
-		(property "Footprint" ""
+		(property "Footprint" "Package_DIP:DIP-24_W15.24mm_Socket"
 			(at 179.07 49.53 0)
 			(hide yes)
@@
 			)
 		)
-		(property "Footprint" ""
+		(property "Footprint" "Package_DIP:DIP-14_W7.62mm_Socket"
 			(at 200.66 129.54 0)
 			(hide yes)
@@
 			)
 		)
-		(property "Footprint" ""
+		(property "Footprint" "Package_DIP:DIP-14_W7.62mm_Socket"
 			(at 200.66 127 0)
 			(hide yes)
@@
 			)
 		)
-		(property "Footprint" ""
+		(property "Footprint" "Package_DIP:DIP-14_W7.62mm_Socket"
 			(at 200.66 132.08 0)
 			(hide yes)
@@
 			)
 		)
-		(property "Footprint" ""
+		(property "Footprint" "Package_DIP:DIP-14_W7.62mm_Socket"
 			(at 200.66 106.68 0)
 			(hide yes)
@@
 			)
 		)
-		(property "Footprint" ""
+		(property "Footprint" "Package_DIP:DIP-14_W7.62mm_Socket"
 			(at 99.06 102.87 0)
 			(hide yes)
@@
 			)
 		)
-		(property "Footprint" ""
+		(property "Footprint" "Package_DIP:DIP-14_W7.62mm_Socket"
 			(at 200.66 104.14 0)
 			(hide yes)
@@
 			)
 		)
-		(property "Footprint" ""
+		(property "Footprint" "Package_DIP:DIP-14_W7.62mm_Socket"
 			(at 200.66 255.27 0)
 			(hide yes)
@@
 			)
 		)
-		(property "Footprint" ""
+		(property "Footprint" "Package_DIP:DIP-14_W7.62mm_Socket"
 			(at 177.8 255.27 0)
 			(hide yes)
@@
 			)
 		)
-		(property "Footprint" ""
+		(property "Footprint" "Package_DIP:DIP-14_W7.62mm_Socket"
 			(at 99.06 171.45 0)
 			(hide yes)
@@
 			)
 		)
-		(property "Footprint" ""
+		(property "Footprint" "Package_DIP:DIP-14_W7.62mm_Socket"
 			(at 200.66 139.7 0)
 			(hide yes)
@@
 			)
 		)
-		(property "Footprint" ""
+		(property "Footprint" "Package_DIP:DIP-14_W7.62mm_Socket"
 			(at 213.36 52.07 0)
 			(hide yes)
@@
 			)
 		)
-		(property "Footprint" ""
+		(property "Footprint" "Package_DIP:DIP-14_W7.62mm_Socket"
 			(at 200.66 121.92 0)
 			(hide yes)
@@
 			)
 		)
-		(property "Footprint" ""
+		(property "Footprint" "Package_DIP:DIP-14_W7.62mm_Socket"
 			(at 200.66 134.62 0)
 			(hide yes)
@@
 			)
 		)
-		(property "Footprint" ""
+		(property "Footprint" "Package_DIP:DIP-14_W7.62mm_Socket"
 			(at 156.21 255.27 0)
 			(hide yes)
