File: schematic/lcd_driver.kicad_sch (KiCad schematic)
At the start: 4 parts, among them U67 74LS573, U69 74LS08

Commit message: feat: address decoding completed, general clean up
Parts:
- renumbered U69 to U100, U67 to U101
Changed lines of the file:
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@@
 		(in_pos_files yes)
 		(dnp no)
-		(property "Reference" "U69"
+		(property "Reference" "U100"
 			(at 169.164 173.736 0)
 			(show_name no)
@@
 			(project "8bit"
 				(path "/ce6ef060-f4bd-4228-ab8d-5cf6f386dba1/0abc0271-e4af-4864-95c9-46cd13d6a322"
-					(reference "U69")
+					(reference "U100")
 					(unit 5)
 				)
@@
 		(dnp no)
 		(fields_autoplaced yes)
-		(property "Reference" "#PWR0179"
+		(property "Reference" "#PWR0264"
 			(at 168.91 74.93 0)
 			(hide yes)
@@
 			(project "8bit"
 				(path "/ce6ef060-f4bd-4228-ab8d-5cf6f386dba1/0abc0271-e4af-4864-95c9-46cd13d6a322"
-					(reference "#PWR0179")
+					(reference "#PWR0264")
 					(unit 1)
 				)
@@
 		(dnp no)
 		(fields_autoplaced yes)
-		(property "Reference" "#PWR0187"
+		(property "Reference" "#PWR0263"
 			(at 161.29 194.31 0)
 			(hide yes)
@@
 			(project "8bit"
 				(path "/ce6ef060-f4bd-4228-ab8d-5cf6f386dba1/0abc0271-e4af-4864-95c9-46cd13d6a322"
-					(reference "#PWR0187")
+					(reference "#PWR0263")
 					(unit 1)
 				)
@@
 		(in_pos_files yes)
 		(dnp no)
-		(property "Reference" "#PWR0184"
+		(property "Reference" "#PWR0261"
 			(at 148.59 87.63 0)
 			(hide yes)
@@
 			(project "8bit"
 				(path "/ce6ef060-f4bd-4228-ab8d-5cf6f386dba1/0abc0271-e4af-4864-95c9-46cd13d6a322"
-					(reference "#PWR0184")
+					(reference "#PWR0261")
 					(unit 1)
 				)
@@
 		(dnp no)
 		(fields_autoplaced yes)
-		(property "Reference" "#PWR0182"
+		(property "Reference" "#PWR0260"
 			(at 123.19 128.27 0)
 			(hide yes)
@@
 			(project "8bit"
 				(path "/ce6ef060-f4bd-4228-ab8d-5cf6f386dba1/0abc0271-e4af-4864-95c9-46cd13d6a322"
-					(reference "#PWR0182")
+					(reference "#PWR0260")
 					(unit 1)
 				)
@@
 		(dnp no)
 		(fields_autoplaced yes)
-		(property "Reference" "#PWR0178"
+		(property "Reference" "#PWR0267"
 			(at 191.77 76.2 0)
 			(hide yes)
@@
 			(project "8bit"
 				(path "/ce6ef060-f4bd-4228-ab8d-5cf6f386dba1/0abc0271-e4af-4864-95c9-46cd13d6a322"
-					(reference "#PWR0178")
+					(reference "#PWR0267")
 					(unit 1)
 				)
@@
 		(dnp no)
 		(fields_autoplaced yes)
-		(property "Reference" "U67"
+		(property "Reference" "U101"
 			(at 125.3333 81.28 0)
 			(show_name no)
@@
 			(project "8bit"
 				(path "/ce6ef060-f4bd-4228-ab8d-5cf6f386dba1/0abc0271-e4af-4864-95c9-46cd13d6a322"
-					(reference "U67")
+					(reference "U101")
 					(unit 1)
 				)
@@
 		(dnp no)
 		(fields_autoplaced yes)
-		(property "Reference" "#PWR0180"
+		(property "Reference" "#PWR0268"
 			(at 191.77 86.36 0)
 			(hide yes)
@@
 			(project "8bit"
 				(path "/ce6ef060-f4bd-4228-ab8d-5cf6f386dba1/0abc0271-e4af-4864-95c9-46cd13d6a322"
-					(reference "#PWR0180")
+					(reference "#PWR0268")
 					(unit 1)
 				)
@@
 		(dnp no)
 		(fields_autoplaced yes)
-		(property "Reference" "#PWR0183"
+		(property "Reference" "#PWR0259"
 			(at 123.19 85.09 0)
 			(hide yes)
@@
 			(project "8bit"
 				(path "/ce6ef060-f4bd-4228-ab8d-5cf6f386dba1/0abc0271-e4af-4864-95c9-46cd13d6a322"
-					(reference "#PWR0183")
+					(reference "#PWR0259")
 					(unit 1)
 				)
@@
 		(dnp no)
 		(fields_autoplaced yes)
-		(property "Reference" "#PWR0188"
+		(property "Reference" "#PWR0262"
 			(at 161.29 166.37 0)
 			(hide yes)
@@
 			(project "8bit"
 				(path "/ce6ef060-f4bd-4228-ab8d-5cf6f386dba1/0abc0271-e4af-4864-95c9-46cd13d6a322"
-					(reference "#PWR0188")
+					(reference "#PWR0262")
 					(unit 1)
 				)
@@
 		(dnp no)
 		(fields_autoplaced yes)
-		(property "Reference" "U69"
+		(property "Reference" "U100"
 			(at 97.7817 102.87 0)
 			(show_name no)
@@
 			(project "8bit"
 				(path "/ce6ef060-f4bd-4228-ab8d-5cf6f386dba1/0abc0271-e4af-4864-95c9-46cd13d6a322"
-					(reference "U69")
+					(reference "U100")
 					(unit 1)
 				)
@@
 		(in_pos_files yes)
 		(dnp no)
-		(property "Reference" "#PWR0181"
+		(property "Reference" "#PWR0266"
 			(at 179.07 86.36 0)
 			(hide yes)
@@
 			(project "8bit"
 				(path "/ce6ef060-f4bd-4228-ab8d-5cf6f386dba1/0abc0271-e4af-4864-95c9-46cd13d6a322"
-					(reference "#PWR0181")
+					(reference "#PWR0266")
 					(unit 1)
 				)
@@
 		(dnp no)
 		(fields_autoplaced yes)
-		(property "Reference" "#PWR0177"
+		(property "Reference" "#PWR0265"
 			(at 168.91 118.11 0)
 			(hide yes)
@@
 			(project "8bit"
 				(path "/ce6ef060-f4bd-4228-ab8d-5cf6f386dba1/0abc0271-e4af-4864-95c9-46cd13d6a322"
-					(reference "#PWR0177")
-					(unit 1)
-				)
+					(reference "#PWR0265")
+					(unit 1)
+				)

Commit message: chore: update bom and footprintss
Parts:
- RV1: footprint (none) -> Resistor_SMD:R_0805_2012Metric
Changed lines of the file:
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@@
 			)
 		)
-		(property "Footprint" ""
+		(property "Footprint" "Resistor_SMD:R_0805_2012Metric"
 			(at 191.77 76.2 0)
 			(hide yes)
