File: schematic/mar.kicad_sch (KiCad schematic)
At the start: 56 parts, among them SW4 SW_DIP_x08, SW9 L/~{H}, U1 74LS04, U2 74LS08, U3 74LS32, U84 74LS161, U85 74LS161, U86 74LS161, U87 74LS161, U88 74LS245, U89 74LS245, U90 74LS245, U91 74LS245

Commit message: feat: address decoding completed, general clean up
Parts:
- renumbered D206 to D1, D190 to D10, D191 to D11, D192 to D12, D193 to D13, D194 to D14, D195 to D15, D196 to D16, D197 to D17, D126 to D2, D127 to D3, D128 to D4, D185 to D5, D186 to D6, D187 to D7, D188 to D8, D189 to D9, R233 to R1, R250 to R10, R210 to R11, R211 to R12, R212 to R13, R213 to R14, R214 to R15, R215 to R16, R216 to R17, R217 to R18, R218 to R19, R232 to R2, R219 to R20, R220 to R21, R221 to R22, R222 to R23, R223 to R24, R224 to R25, R225 to R26, R234 to R3, R235 to R4, R236 to R5, R237 to R6, R238 to R7, R239 to R8, R6 to R9, SW4 to SW1, SW9 to SW2, U90 to U1, U88 to U10, U89 to U11, U91 to U2, U1 to U3, U2 to U4, U3 to U4, U3 to U5, U84 to U6, U85 to U7, U86 to U8, U87 to U9

Commit message: chore: update bom and footprintss
Parts:
- R9: footprint (none) -> Resistor_SMD:R_0805_2012Metric
- U1, U2: footprint (none) -> Package_DIP:DIP-20_W7.62mm_Socket
- U3, U4, U5: footprint (none) -> Package_DIP:DIP-14_W7.62mm_Socket
Changed lines of the file:
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@@
 			)
 		)
-		(property "Footprint" ""
+		(property "Footprint" "Package_DIP:DIP-14_W7.62mm_Socket"
 			(at 139.7 227.33 0)
 			(hide yes)
@@
 			)
 		)
-		(property "Footprint" ""
+		(property "Footprint" "Package_DIP:DIP-14_W7.62mm_Socket"
 			(at 359.41 271.78 0)
 			(hide yes)
@@
 			)
 		)
-		(property "Footprint" ""
+		(property "Footprint" "Package_DIP:DIP-14_W7.62mm_Socket"
 			(at 236.22 161.29 0)
 			(hide yes)
@@
 			)
 		)
-		(property "Footprint" ""
+		(property "Footprint" "Package_DIP:DIP-14_W7.62mm_Socket"
 			(at 214.63 163.83 0)
 			(hide yes)
@@
 			)
 		)
-		(property "Footprint" ""
+		(property "Footprint" "Package_DIP:DIP-20_W7.62mm_Socket"
 			(at 93.98 132.08 0)
 			(hide yes)
@@
 			)
 		)
-		(property "Footprint" ""
+		(property "Footprint" "Package_DIP:DIP-14_W7.62mm_Socket"
 			(at 379.73 271.78 0)
 			(hide yes)
@@
 			)
 		)
-		(property "Footprint" ""
+		(property "Footprint" "Package_DIP:DIP-14_W7.62mm_Socket"
 			(at 237.49 267.97 0)
 			(hide yes)
@@
 			)
 		)
-		(property "Footprint" ""
+		(property "Footprint" "Package_DIP:DIP-14_W7.62mm_Socket"
 			(at 457.2 111.76 0)
 			(hide yes)
@@
 			)
 		)
-		(property "Footprint" ""
+		(property "Footprint" "Package_DIP:DIP-14_W7.62mm_Socket"
 			(at 198.12 273.05 0)
 			(hide yes)
@@
 			)
 		)
-		(property "Footprint" ""
+		(property "Footprint" "Package_DIP:DIP-20_W7.62mm_Socket"
 			(at 138.43 165.1 0)
 			(hide yes)
@@
 			)
 		)
-		(property "Footprint" ""
+		(property "Footprint" "Resistor_SMD:R_0805_2012Metric"
 			(at 109.982 252.73 90)
 			(hide yes)
@@
 			)
 		)
-		(property "Footprint" ""
+		(property "Footprint" "Package_DIP:DIP-14_W7.62mm_Socket"
 			(at 400.05 271.78 0)
 			(hide yes)
@@
 			)
 		)
-		(property "Footprint" ""
+		(property "Footprint" "Package_DIP:DIP-14_W7.62mm_Socket"
 			(at 215.9 270.51 0)
 			(hide yes)
