File: schematic/misc.kicad_sch (KiCad schematic)
At the start: 10 parts, among them SW6 SW_SPDT, SW7 RESET, U103 74LS04

Commit message: feat: address decoding completed, general clean up
Parts:
- renumbered D1 to D191, D2 to D192, R5 to R238, R3 to R239, R1 to R240, R2 to R241, R4 to R242, SW6 to SW8, U103 to U111
Changed lines of the file:
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@@
 		(dnp no)
 		(fields_autoplaced yes)
-		(property "Reference" "R2"
+		(property "Reference" "R241"
 			(at 71.12 63.4999 0)
 			(show_name no)
@@
 			(project "8bit"
 				(path "/ce6ef060-f4bd-4228-ab8d-5cf6f386dba1/ecff370d-b3fa-44b6-a1ec-dd8706389b07"
-					(reference "R2")
+					(reference "R241")
 					(unit 1)
 				)
@@
 		(dnp no)
 		(fields_autoplaced yes)
-		(property "Reference" "#PWR05"
+		(property "Reference" "#PWR0294"
 			(at 160.02 168.91 0)
 			(hide yes)
@@
 			(project "8bit"
 				(path "/ce6ef060-f4bd-4228-ab8d-5cf6f386dba1/ecff370d-b3fa-44b6-a1ec-dd8706389b07"
-					(reference "#PWR05")
+					(reference "#PWR0294")
 					(unit 1)
 				)
@@
 		(dnp no)
 		(fields_autoplaced yes)
-		(property "Reference" "R3"
+		(property "Reference" "R239"
 			(at 52.07 58.4199 0)
 			(show_name no)
@@
 			(project "8bit"
 				(path "/ce6ef060-f4bd-4228-ab8d-5cf6f386dba1/ecff370d-b3fa-44b6-a1ec-dd8706389b07"
-					(reference "R3")
+					(reference "R239")
 					(unit 1)
 				)
@@
 		(dnp no)
 		(fields_autoplaced yes)
-		(property "Reference" "U103"
+		(property "Reference" "U111"
 			(at 71.12 86.36 0)
 			(show_name no)
@@
 			(project "8bit"
 				(path "/ce6ef060-f4bd-4228-ab8d-5cf6f386dba1/ecff370d-b3fa-44b6-a1ec-dd8706389b07"
-					(reference "U103")
+					(reference "U111")
 					(unit 1)
 				)
@@
 		(dnp no)
 		(fields_autoplaced yes)
-		(property "Reference" "#PWR01"
+		(property "Reference" "#PWR0292"
 			(at 63.5 41.91 0)
 			(hide yes)
@@
 			(project "8bit"
 				(path "/ce6ef060-f4bd-4228-ab8d-5cf6f386dba1/ecff370d-b3fa-44b6-a1ec-dd8706389b07"
-					(reference "#PWR01")
+					(reference "#PWR0292")
 					(unit 1)
 				)
@@
 		(dnp no)
 		(fields_autoplaced yes)
-		(property "Reference" "R4"
+		(property "Reference" "R242"
 			(at 80.01 58.4199 0)
 			(show_name no)
@@
 			(project "8bit"
 				(path "/ce6ef060-f4bd-4228-ab8d-5cf6f386dba1/ecff370d-b3fa-44b6-a1ec-dd8706389b07"
-					(reference "R4")
+					(reference "R242")
 					(unit 1)
 				)
@@
 		(dnp no)
 		(fields_autoplaced yes)
-		(property "Reference" "U103"
+		(property "Reference" "U111"
 			(at 166.37 176.5299 0)
 			(show_name no)
@@
 			(project "8bit"
 				(path "/ce6ef060-f4bd-4228-ab8d-5cf6f386dba1/ecff370d-b3fa-44b6-a1ec-dd8706389b07"
-					(reference "U103")
+					(reference "U111")
 					(unit 7)
 				)
@@
 		(dnp no)
 		(fields_autoplaced yes)
-		(property "Reference" "D1"
+		(property "Reference" "D191"
 			(at 60.96 55.8799 90)
 			(show_name no)
@@
 			(project "8bit"
 				(path "/ce6ef060-f4bd-4228-ab8d-5cf6f386dba1/ecff370d-b3fa-44b6-a1ec-dd8706389b07"
-					(reference "D1")
+					(reference "D191")
 					(unit 1)
 				)
@@
 		(dnp no)
 		(fields_autoplaced yes)
-		(property "Reference" "D2"
+		(property "Reference" "D192"
 			(at 71.12 55.8799 90)
 			(show_name no)
@@
 			(project "8bit"
 				(path "/ce6ef060-f4bd-4228-ab8d-5cf6f386dba1/ecff370d-b3fa-44b6-a1ec-dd8706389b07"
-					(reference "D2")
+					(reference "D192")
 					(unit 1)
 				)
@@
 		(dnp no)
 		(fields_autoplaced yes)
-		(property "Reference" "#PWR02"
+		(property "Reference" "#PWR0293"
 			(at 63.5 74.93 0)
 			(hide yes)
@@
 			(project "8bit"
 				(path "/ce6ef060-f4bd-4228-ab8d-5cf6f386dba1/ecff370d-b3fa-44b6-a1ec-dd8706389b07"
-					(reference "#PWR02")
+					(reference "#PWR0293")
 					(unit 1)
 				)
@@
 		(dnp no)
 		(fields_autoplaced yes)
-		(property "Reference" "SW6"
+		(property "Reference" "SW8"
 			(at 68.58 45.7199 90)
 			(show_name no)
@@
 			(project "8bit"
 				(path "/ce6ef060-f4bd-4228-ab8d-5cf6f386dba1/ecff370d-b3fa-44b6-a1ec-dd8706389b07"
-					(reference "SW6")
+					(reference "SW8")
 					(unit 1)
 				)
@@
 		(in_pos_files yes)
 		(dnp no)
-		(property "Reference" "R5"
+		(property "Reference" "R238"
 			(at 45.72 97.7899 0)
 			(show_name no)
@@
 			(project "8bit"
 				(path "/ce6ef060-f4bd-4228-ab8d-5cf6f386dba1/ecff370d-b3fa-44b6-a1ec-dd8706389b07"
-					(reference "R5")
+					(reference "R238")
 					(unit 1)
 				)
@@
 		(dnp no)
 		(fields_autoplaced yes)
-		(property "Reference" "#PWR03"
+		(property "Reference" "#PWR0291"
 			(at 58.42 111.76 0)
 			(hide yes)
@@
 			(project "8bit"
 				(path "/ce6ef060-f4bd-4228-ab8d-5cf6f386dba1/ecff370d-b3fa-44b6-a1ec-dd8706389b07"
-					(reference "#PWR03")
+					(reference "#PWR0291")
 					(unit 1)
 				)
@@
 		(dnp no)
 		(fields_autoplaced yes)
-		(property "Reference" "R1"
+		(property "Reference" "R240"
 			(at 60.96 63.4999 0)
 			(show_name no)
@@
 			(project "8bit"
 				(path "/ce6ef060-f4bd-4228-ab8d-5cf6f386dba1/ecff370d-b3fa-44b6-a1ec-dd8706389b07"
-					(reference "R1")
+					(reference "R240")
 					(unit 1)
 				)
@@
 		(dnp no)
 		(fields_autoplaced yes)
-		(property "Reference" "#PWR04"
+		(property "Reference" "#PWR0290"
 			(at 48.26 99.06 0)
 			(hide yes)
@@
 			(project "8bit"
 				(path "/ce6ef060-f4bd-4228-ab8d-5cf6f386dba1/ecff370d-b3fa-44b6-a1ec-dd8706389b07"
-					(reference "#PWR04")
+					(reference "#PWR0290")
 					(unit 1)
 				)
@@
 		(dnp no)
 		(fields_autoplaced yes)
-		(property "Reference" "#PWR06"
+		(property "Reference" "#PWR0295"
 			(at 160.02 196.85 0)
 			(hide yes)
@@
 			(project "8bit"
 				(path "/ce6ef060-f4bd-4228-ab8d-5cf6f386dba1/ecff370d-b3fa-44b6-a1ec-dd8706389b07"
-					(reference "#PWR06")
-					(unit 1)
-				)
+					(reference "#PWR0295")
+					(unit 1)
+				)

Commit message: chore: update bom and footprintss
Parts:
- R238, R239, R240, R241, R242: footprint (none) -> Resistor_SMD:R_0805_2012Metric
- U111: footprint (none) -> Package_DIP:DIP-14_W7.62mm_Socket
Changed lines of the file:
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@@
 			)
 		)
-		(property "Footprint" ""
+		(property "Footprint" "Resistor_SMD:R_0805_2012Metric"
 			(at 66.802 64.77 90)
 			(hide yes)
@@
 			)
 		)
-		(property "Footprint" ""
+		(property "Footprint" "Resistor_SMD:R_0805_2012Metric"
 			(at 47.752 59.69 90)
 			(hide yes)
@@
 			)
 		)
-		(property "Footprint" ""
+		(property "Footprint" "Package_DIP:DIP-14_W7.62mm_Socket"
 			(at 71.12 95.25 0)
 			(hide yes)
@@
 			)
 		)
-		(property "Footprint" ""
+		(property "Footprint" "Resistor_SMD:R_0805_2012Metric"
 			(at 75.692 59.69 90)
 			(hide yes)
@@
 			)
 		)
-		(property "Footprint" ""
+		(property "Footprint" "Package_DIP:DIP-14_W7.62mm_Socket"
 			(at 160.02 177.8 0)
 			(hide yes)
@@
 			)
 		)
-		(property "Footprint" ""
+		(property "Footprint" "Resistor_SMD:R_0805_2012Metric"
 			(at 50.038 99.06 90)
 			(hide yes)
@@
 			)
 		)
-		(property "Footprint" ""
+		(property "Footprint" "Resistor_SMD:R_0805_2012Metric"
 			(at 56.642 64.77 90)
 			(hide yes)
