File: schematic/ram.kicad_sch (KiCad schematic)
At the start: 30 parts, among them SW5 SW_DIP_x08, U19 HM62256BLP, U20 74LS245, U4 74LS02, U94 74LS245, U95 74LS08

Commit message: feat: address decoding completed, general clean up
Parts:
- renumbered D49 to D69, D50 to D70, D51 to D71, D52 to D72, D53 to D73, D54 to D74, D55 to D75, D56 to D76, R246 to R100, R247 to R101, R49 to R102, R50 to R103, R51 to R104, R52 to R105, R53 to R106, R54 to R107, R55 to R108, R56 to R109, R240 to R94, R241 to R95, R242 to R96, R243 to R97, R244 to R98, R245 to R99, SW5 to SW3, U95 to U30, U4 to U31, U19 to U32, U94 to U33, U20 to U34

Commit message: chore: update bom and footprintss
Parts:
- U30, U31: footprint (none) -> Package_DIP:DIP-14_W7.62mm_Socket
Changed lines of the file:
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@@
 			)
 		)
-		(property "Footprint" ""
+		(property "Footprint" "Package_DIP:DIP-14_W7.62mm_Socket"
 			(at 54.61 114.3 0)
 			(hide yes)
@@
 			)
 		)
-		(property "Footprint" ""
+		(property "Footprint" "Package_DIP:DIP-14_W7.62mm_Socket"
 			(at 45.72 175.26 0)
 			(hide yes)
@@
 			)
 		)
-		(property "Footprint" ""
+		(property "Footprint" "Package_DIP:DIP-14_W7.62mm_Socket"
 			(at 54.61 137.16 0)
 			(hide yes)
@@
 			)
 		)
-		(property "Footprint" ""
+		(property "Footprint" "Package_DIP:DIP-14_W7.62mm_Socket"
 			(at 74.93 175.26 0)
 			(hide yes)
@@
 			)
 		)
-		(property "Footprint" ""
+		(property "Footprint" "Package_DIP:DIP-14_W7.62mm_Socket"
 			(at 69.85 101.6 0)
 			(hide yes)
@@
 			)
 		)
-		(property "Footprint" ""
+		(property "Footprint" "Package_DIP:DIP-14_W7.62mm_Socket"
 			(at 69.85 125.73 0)
 			(hide yes)
@@
 			)
 		)
-		(property "Footprint" ""
+		(property "Footprint" "Package_DIP:DIP-14_W7.62mm_Socket"
 			(at 36.83 125.73 0)
 			(hide yes)
