File: schematic/register_h_l.kicad_sch (KiCad schematic)
At the start: 40 parts, among them U26 74LS193, U27 74LS193, U48 74LS193, U49 74LS193, U50 74LS245, U51 74LS245, U52 74LS245, U53 74LS245

Commit message: feat: address decoding completed, general clean up
Parts:
- added U41: 74LS00, symbol 74xx:74LS00
- renumbered D165 to D102, D173 to D103, D166 to D104, D174 to D105, D167 to D106, D175 to D107, D168 to D108, D176 to D109, D169 to D110, D177 to D111, D170 to D112, D178 to D113, D171 to D114, D179 to D115, D172 to D116, D180 to D117, R181 to R137, R189 to R138, R182 to R139, R190 to R140, R183 to R141, R191 to R142, R184 to R143, R192 to R144, R185 to R145, R193 to R146, R186 to R147, R194 to R148, R187 to R149, R195 to R150, R188 to R151, R196 to R152, U26 to U42, U27 to U43, U48 to U44, U49 to U45, U50 to U46, U51 to U47, U52 to U48, U53 to U49
Connections:
- net +5V: now also U41.14 (VCC)
- net GND: now also U41.7 (GND)
- net ~{REG_H_I}: no longer names the net of U44.11 (~{LOAD}), U45.11 (~{LOAD})
- net ~{REG_H_I}: now also U41.6
- net ~{REG_L_I}: no longer names the net of U42.11 (~{LOAD}), U43.11 (~{LOAD})
- net ~{REG_L_I}: now also U41.3
- new net CLK: U41.1, U41.4
- new net REG_H_I: U41.5
- new net REG_L_I: U41.2
- no-connect marks 0 -> 2

Commit message: chore: update bom and footprintss
Parts:
- U41: footprint (none) -> Package_DIP:DIP-14_W7.62mm_Socket
Changed lines of the file:
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@@
 			)
 		)
-		(property "Footprint" ""
+		(property "Footprint" "Package_DIP:DIP-14_W7.62mm_Socket"
 			(at 29.21 87.63 0)
 			(hide yes)
@@
 			)
 		)
-		(property "Footprint" ""
+		(property "Footprint" "Package_DIP:DIP-14_W7.62mm_Socket"
 			(at 30.48 195.58 0)
 			(hide yes)
@@
 			)
 		)
-		(property "Footprint" ""
+		(property "Footprint" "Package_DIP:DIP-14_W7.62mm_Socket"
 			(at 191.77 259.08 0)
 			(hide yes)
