File: schematic/stack_pointer.kicad_sch (KiCad schematic)
At the start: 39 parts, among them U11 74LS193, U12 74LS193, U13 74LS193, U14 74LS193, U15 74LS245, U16 74LS245, U92 74LS00

Commit message: chore: sync outdated schematic files
Connections:
- net ~{SP_L_I} renamed SP_L_I
Changed lines of the file:
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@@
 		)
 	)
-	(hierarchical_label "~{SP_L_I}"
+	(hierarchical_label "SP_L_I"
 		(shape input)
 		(at 69.85 72.39 180)

Commit message: feat: address decoding completed, general clean up
Parts:
- renumbered D33 to D34, D34 to D35, D35 to D36, D36 to D37, D37 to D38, D38 to D39, D39 to D40, D40 to D41, D41 to D42, D42 to D43, D43 to D44, D44 to D45, D45 to D46, D46 to D47, D47 to D48, D48 to D49, R33 to R43, R34 to R44, R35 to R45, R36 to R46, R37 to R47, R38 to R48, R39 to R49, R40 to R50, R41 to R51, R42 to R52, R43 to R53, R44 to R54, R45 to R55, R46 to R56, R47 to R57, R48 to R58, U92 to U20, U11 to U21, U12 to U22, U13 to U23, U14 to U24, U15 to U25, U16 to U26
Connections:
- no-connect marks 0 -> 2

Commit message: chore: update bom and footprintss
Parts:
- U20: footprint (none) -> Package_DIP:DIP-14_W7.62mm_Socket
Changed lines of the file:
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@@
 			)
 		)
-		(property "Footprint" ""
+		(property "Footprint" "Package_DIP:DIP-14_W7.62mm_Socket"
 			(at 77.47 74.93 0)
 			(hide yes)
@@
 			)
 		)
-		(property "Footprint" ""
+		(property "Footprint" "Package_DIP:DIP-14_W7.62mm_Socket"
 			(at 198.12 167.64 0)
 			(hide yes)
@@
 			)
 		)
-		(property "Footprint" ""
+		(property "Footprint" "Package_DIP:DIP-14_W7.62mm_Socket"
 			(at 73.66 180.34 0)
 			(hide yes)
