File: schematic/step_counter.kicad_sch (KiCad schematic)
At the start: 11 parts, among them U102 74LS00, U61 74LS161, U62 74LS02

Commit message: feat: address decoding completed, general clean up
Parts:
- renumbered D181 to D178, D182 to D179, D183 to D180, D184 to D181, R201 to R219, R204 to R220, R205 to R221, R206 to R222, U102 to U86, U62 to U87, U61 to U88
Changed lines of the file:
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@@
 		(in_pos_files yes)
 		(dnp no)
-		(property "Reference" "#PWR0166"
+		(property "Reference" "#PWR0235"
 			(at 158.75 195.58 0)
 			(hide yes)
@@
 			(project "8bit"
 				(path "/ce6ef060-f4bd-4228-ab8d-5cf6f386dba1/b16f9325-fb3f-40a8-8bed-2a1940a96351"
-					(reference "#PWR0166")
+					(reference "#PWR0235")
 					(unit 1)
 				)
@@
 		(in_pos_files yes)
 		(dnp no)
-		(property "Reference" "R201"
+		(property "Reference" "R219"
 			(at 161.798 85.09 90)
 			(show_name no)
@@
 			(project "8bit"
 				(path "/ce6ef060-f4bd-4228-ab8d-5cf6f386dba1/b16f9325-fb3f-40a8-8bed-2a1940a96351"
-					(reference "R201")
+					(reference "R219")
 					(unit 1)
 				)
@@
 		(in_pos_files yes)
 		(dnp no)
-		(property "Reference" "D183"
+		(property "Reference" "D180"
 			(at 171.958 90.17 0)
 			(show_name no)
@@
 			(project "8bit"
 				(path "/ce6ef060-f4bd-4228-ab8d-5cf6f386dba1/b16f9325-fb3f-40a8-8bed-2a1940a96351"
-					(reference "D183")
+					(reference "D180")
 					(unit 1)
 				)
@@
 		(dnp no)
 		(fields_autoplaced yes)
-		(property "Reference" "U102"
+		(property "Reference" "U86"
 			(at 144.78 175.2599 0)
 			(show_name no)
@@
 			(project "8bit"
 				(path "/ce6ef060-f4bd-4228-ab8d-5cf6f386dba1/b16f9325-fb3f-40a8-8bed-2a1940a96351"
-					(reference "U102")
+					(reference "U86")
 					(unit 5)
 				)
@@
 		(dnp no)
 		(fields_autoplaced yes)
-		(property "Reference" "U102"
+		(property "Reference" "U86"
 			(at 76.1917 78.74 0)
 			(show_name no)
@@
 			(project "8bit"
 				(path "/ce6ef060-f4bd-4228-ab8d-5cf6f386dba1/b16f9325-fb3f-40a8-8bed-2a1940a96351"
-					(reference "U102")
+					(reference "U86")
 					(unit 2)
 				)
@@
 		(dnp no)
 		(fields_autoplaced yes)
-		(property "Reference" "U102"
+		(property "Reference" "U86"
 			(at 54.6017 78.74 0)
 			(show_name no)
@@
 			(project "8bit"
 				(path "/ce6ef060-f4bd-4228-ab8d-5cf6f386dba1/b16f9325-fb3f-40a8-8bed-2a1940a96351"
-					(reference "U102")
+					(reference "U86")
 					(unit 3)
 				)
@@
 		(in_pos_files yes)
 		(dnp no)
-		(property "Reference" "D181"
+		(property "Reference" "D178"
 			(at 161.798 90.17 0)
 			(show_name no)
@@
 			(project "8bit"
 				(path "/ce6ef060-f4bd-4228-ab8d-5cf6f386dba1/b16f9325-fb3f-40a8-8bed-2a1940a96351"
-					(reference "D181")
+					(reference "D178")
 					(unit 1)
 				)
@@
 		(dnp no)
 		(fields_autoplaced yes)
-		(property "Reference" "U62"
+		(property "Reference" "U87"
 			(at 144.78 123.19 0)
 			(show_name no)
@@
 			(project "8bit"
 				(path "/ce6ef060-f4bd-4228-ab8d-5cf6f386dba1/b16f9325-fb3f-40a8-8bed-2a1940a96351"
-					(reference "U62")
+					(reference "U87")
 					(unit 4)
 				)
@@
 		(in_pos_files yes)
 		(dnp no)
-		(property "Reference" "U62"
+		(property "Reference" "U87"
 			(at 130.81 122.936 0)
 			(show_name no)
@@
 			(project "8bit"
 				(path "/ce6ef060-f4bd-4228-ab8d-5cf6f386dba1/b16f9325-fb3f-40a8-8bed-2a1940a96351"
-					(reference "U62")
+					(reference "U87")
 					(unit 3)
 				)
@@
 		(in_pos_files yes)
 		(dnp no)
-		(property "Reference" "#PWR0165"
+		(property "Reference" "#PWR0236"
 			(at 171.45 104.14 0)
 			(hide yes)
@@
 			(project "8bit"
 				(path "/ce6ef060-f4bd-4228-ab8d-5cf6f386dba1/b16f9325-fb3f-40a8-8bed-2a1940a96351"
-					(reference "#PWR0165")
+					(reference "#PWR0236")
 					(unit 1)
 				)
@@
 		(in_pos_files yes)
 		(dnp no)
-		(property "Reference" "U102"
+		(property "Reference" "U86"
 			(at 109.728 141.986 0)
 			(show_name no)
@@
 			(project "8bit"
 				(path "/ce6ef060-f4bd-4228-ab8d-5cf6f386dba1/b16f9325-fb3f-40a8-8bed-2a1940a96351"
-					(reference "U102")
+					(reference "U86")
 					(unit 4)
 				)
@@
 		(dnp no)
 		(fields_autoplaced yes)
-		(property "Reference" "#PWR0163"
+		(property "Reference" "#PWR0230"
 			(at 129.54 63.5 0)
 			(hide yes)
@@
 			(project "8bit"
 				(path "/ce6ef060-f4bd-4228-ab8d-5cf6f386dba1/b16f9325-fb3f-40a8-8bed-2a1940a96351"
-					(reference "#PWR0163")
+					(reference "#PWR0230")
 					(unit 1)
 				)
@@
 		(in_pos_files yes)
 		(dnp no)
-		(property "Reference" "R205"
+		(property "Reference" "R221"
 			(at 171.958 85.09 90)
 			(show_name no)
@@
 			(project "8bit"
 				(path "/ce6ef060-f4bd-4228-ab8d-5cf6f386dba1/b16f9325-fb3f-40a8-8bed-2a1940a96351"
-					(reference "R205")
+					(reference "R221")
 					(unit 1)
 				)
@@
 		(in_pos_files yes)
 		(dnp no)
-		(property "Reference" "D182"
+		(property "Reference" "D179"
 			(at 166.878 90.17 0)
 			(show_name no)
@@
 			(project "8bit"
 				(path "/ce6ef060-f4bd-4228-ab8d-5cf6f386dba1/b16f9325-fb3f-40a8-8bed-2a1940a96351"
-					(reference "D182")
+					(reference "D179")
 					(unit 1)
 				)
@@
 		(in_pos_files yes)
 		(dnp no)
-		(property "Reference" "R204"
+		(property "Reference" "R220"
 			(at 166.878 85.09 90)
 			(show_name no)
@@
 			(project "8bit"
 				(path "/ce6ef060-f4bd-4228-ab8d-5cf6f386dba1/b16f9325-fb3f-40a8-8bed-2a1940a96351"
-					(reference "R204")
+					(reference "R220")
 					(unit 1)
 				)
@@
 		(dnp no)
 		(fields_autoplaced yes)
-		(property "Reference" "U61"
+		(property "Reference" "U88"
 			(at 131.6833 59.69 0)
 			(show_name no)
@@
 			(project "8bit"
 				(path "/ce6ef060-f4bd-4228-ab8d-5cf6f386dba1/b16f9325-fb3f-40a8-8bed-2a1940a96351"
-					(reference "U61")
+					(reference "U88")
 					(unit 1)
 				)
@@
 		(dnp no)
 		(fields_autoplaced yes)
-		(property "Reference" "U62"
+		(property "Reference" "U87"
 			(at 165.1 175.2599 0)
 			(show_name no)
@@
 			(project "8bit"
 				(path "/ce6ef060-f4bd-4228-ab8d-5cf6f386dba1/b16f9325-fb3f-40a8-8bed-2a1940a96351"
-					(reference "U62")
+					(reference "U87")
 					(unit 5)
 				)
@@
 		(dnp no)
 		(fields_autoplaced yes)
-		(property "Reference" "#PWR0168"
+		(property "Reference" "#PWR0234"
 			(at 158.75 167.64 0)
 			(hide yes)
@@
 			(project "8bit"
 				(path "/ce6ef060-f4bd-4228-ab8d-5cf6f386dba1/b16f9325-fb3f-40a8-8bed-2a1940a96351"
-					(reference "#PWR0168")
+					(reference "#PWR0234")
 					(unit 1)
 				)
@@
 		(dnp no)
 		(fields_autoplaced yes)
-		(property "Reference" "U102"
+		(property "Reference" "U86"
 			(at 97.7817 78.74 0)
 			(show_name no)
@@
 			(project "8bit"
 				(path "/ce6ef060-f4bd-4228-ab8d-5cf6f386dba1/b16f9325-fb3f-40a8-8bed-2a1940a96351"
-					(reference "U102")
+					(reference "U86")
 					(unit 1)
 				)
@@
 		(in_pos_files yes)
 		(dnp no)
-		(property "Reference" "#PWR0279"
+		(property "Reference" "#PWR0233"
 			(at 138.43 195.58 0)
 			(hide yes)
@@
 			(project "8bit"
 				(path "/ce6ef060-f4bd-4228-ab8d-5cf6f386dba1/b16f9325-fb3f-40a8-8bed-2a1940a96351"
-					(reference "#PWR0279")
+					(reference "#PWR0233")
 					(unit 1)
 				)
@@
 		(dnp no)
 		(fields_autoplaced yes)
-		(property "Reference" "U62"
+		(property "Reference" "U87"
 			(at 95.25 123.19 0)
 			(show_name no)
@@
 			(project "8bit"
 				(path "/ce6ef060-f4bd-4228-ab8d-5cf6f386dba1/b16f9325-fb3f-40a8-8bed-2a1940a96351"
-					(reference "U62")
+					(reference "U87")
 					(unit 1)
 				)
@@
 		(dnp no)
 		(fields_autoplaced yes)
-		(property "Reference" "U62"
+		(property "Reference" "U87"
 			(at 110.49 123.19 0)
 			(show_name no)
@@
 			(project "8bit"
 				(path "/ce6ef060-f4bd-4228-ab8d-5cf6f386dba1/b16f9325-fb3f-40a8-8bed-2a1940a96351"
-					(reference "U62")
+					(reference "U87")
 					(unit 2)
 				)
@@
 		(in_pos_files yes)
 		(dnp no)
-		(property "Reference" "R206"
+		(property "Reference" "R222"
 			(at 177.038 85.09 90)
 			(show_name no)
@@
 			(project "8bit"
 				(path "/ce6ef060-f4bd-4228-ab8d-5cf6f386dba1/b16f9325-fb3f-40a8-8bed-2a1940a96351"
-					(reference "R206")
+					(reference "R222")
 					(unit 1)
 				)
@@
 		(in_pos_files yes)
 		(dnp no)
-		(property "Reference" "#PWR0167"
+		(property "Reference" "#PWR0229"
 			(at 109.22 82.55 0)
 			(hide yes)
@@
 			(project "8bit"
 				(path "/ce6ef060-f4bd-4228-ab8d-5cf6f386dba1/b16f9325-fb3f-40a8-8bed-2a1940a96351"
-					(reference "#PWR0167")
+					(reference "#PWR0229")
 					(unit 1)
 				)
@@
 		(dnp no)
 		(fields_autoplaced yes)
-		(property "Reference" "#PWR0278"
+		(property "Reference" "#PWR0232"
 			(at 138.43 167.64 0)
 			(hide yes)
@@
 			(project "8bit"
 				(path "/ce6ef060-f4bd-4228-ab8d-5cf6f386dba1/b16f9325-fb3f-40a8-8bed-2a1940a96351"
-					(reference "#PWR0278")
+					(reference "#PWR0232")
 					(unit 1)
 				)
@@
 		(in_pos_files yes)
 		(dnp no)
-		(property "Reference" "#PWR0164"
+		(property "Reference" "#PWR0231"
 			(at 129.54 106.68 0)
 			(hide yes)
@@
 			(project "8bit"
 				(path "/ce6ef060-f4bd-4228-ab8d-5cf6f386dba1/b16f9325-fb3f-40a8-8bed-2a1940a96351"
-					(reference "#PWR0164")
+					(reference "#PWR0231")
 					(unit 1)
 				)
@@
 		(in_pos_files yes)
 		(dnp no)
-		(property "Reference" "D184"
+		(property "Reference" "D181"
 			(at 177.038 90.17 0)
 			(show_name no)
@@
 			(project "8bit"
 				(path "/ce6ef060-f4bd-4228-ab8d-5cf6f386dba1/b16f9325-fb3f-40a8-8bed-2a1940a96351"
-					(reference "D184")
+					(reference "D181")
 					(unit 1)
 				)

Commit message: chore: update bom and footprintss
Parts:
- U86: footprint (none) -> Package_DIP:DIP-14_W7.62mm_Socket
Changed lines of the file:
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@@
 			)
 		)
-		(property "Footprint" ""
+		(property "Footprint" "Package_DIP:DIP-14_W7.62mm_Socket"
 			(at 138.43 176.53 0)
 			(hide yes)
@@
 			)
 		)
-		(property "Footprint" ""
+		(property "Footprint" "Package_DIP:DIP-14_W7.62mm_Socket"
 			(at 76.2 87.63 0)
 			(hide yes)
@@
 			)
 		)
-		(property "Footprint" ""
+		(property "Footprint" "Package_DIP:DIP-14_W7.62mm_Socket"
 			(at 54.61 87.63 0)
 			(hide yes)
@@
 			)
 		)
-		(property "Footprint" ""
+		(property "Footprint" "Package_DIP:DIP-14_W7.62mm_Socket"
 			(at 110.49 135.89 0)
 			(hide yes)
@@
 			)
 		)
-		(property "Footprint" ""
+		(property "Footprint" "Package_DIP:DIP-14_W7.62mm_Socket"
 			(at 97.79 87.63 0)
 			(hide yes)
